File: pcb/OPS.sch (KiCad schematic (older format))
At the start: 45 parts, among them P10 2SC3281, P11 2SA1302, P6 MJE350, P7 MJE340, P8 2SA1302, P9 2SC3281, Q13 MPSA56_PNP_EBC, Q14 MPSA06_NPN_EBC, Q15 MPSA56_PNP_EBC, Q16 MPSA06_NPN_EBC, Q17 MJE340_NPN_ECB, Q18 MJE350_PNP_EBC, Q19 MJE340_NPN_ECB, Q20 MJE350_PNP_EBC

Commit message: Cambio footprints, empiezo a re-rutear
Parts:
- P10: renamed from P9; footprint Pin_Headers:Pin_Header_Straight_1x03 -> pcb:bornera_grande
- P11: renamed from P10; footprint Pin_Headers:Pin_Header_Straight_1x03 -> pcb:bornera_grande
- P12: renamed from P11; footprint Pin_Headers:Pin_Header_Straight_1x03 -> pcb:bornera_grande
- P9: renamed from P8; footprint Pin_Headers:Pin_Header_Straight_1x03 -> pcb:bornera_grande
- Q13, Q14, Q15, Q16: footprint Transistors_TO-220:TO-220_Neutral123_Vertical -> pcb:MPSA06-56_TO92_EBC
- Q19: footprint Transistors_TO-220:TO-220_Neutral123_Vertical -> pcb:MJE340_gclass
- Q20: footprint Transistors_TO-220:TO-220_Neutral123_Vertical -> pcb:MJE_350_gclass
- R27, R28: footprint Resistors_ThroughHole:Resistor_Ceramic_Horizontal_L23mm-W9mm-H9mm-p30mm -> pcb:RESIST_35MMX10MM
- renumbered P6 to P7, P7 to P8
Changed lines of the file:
@@
 F 0 "Q13" H 3600 1400 50  0000 R CNN
 F 1 "MPSA56_PNP_EBC" H 3700 1100 50  0000 R CNN
-F 2 "Transistors_TO-220:TO-220_Neutral123_Vertical" H 3500 1450 29  0001 C CNN
+F 2 "pcb:MPSA06-56_TO92_EBC" H 3500 1450 29  0001 C CNN
 F 3 "" H 3300 1350 60  0000 C CNN
 	1    3300 1350
@@
 F 0 "Q15" H 4200 1400 50  0000 R CNN
 F 1 "MPSA56_PNP_EBC" H 4350 1100 50  0000 R CNN
-F 2 "Transistors_TO-220:TO-220_Neutral123_Vertical" H 4100 1450 29  0001 C CNN
+F 2 "pcb:MPSA06-56_TO92_EBC" H 4100 1450 29  0001 C CNN
 F 3 "" H 3900 1350 60  0000 C CNN
 	1    3900 1350
@@
 F 0 "Q19" H 5550 1900 50  0000 R CNN
 F 1 "MJE340_NPN_ECB" H 5700 2100 50  0000 R CNN
-F 2 "Transistors_TO-220:TO-220_Neutral123_Vertical" H 5450 1950 29  0001 C CNN
+F 2 "pcb:MJE340_gclass" H 5450 1950 29  0001 C CNN
 F 3 "" H 5250 1850 60  0000 C CNN
 	1    5250 1850
@@
 F 0 "R27" V 6030 3300 50  0000 C CNN
 F 1 "R" V 5950 3300 50  0000 C CNN
-F 2 "Resistors_ThroughHole:Resistor_Ceramic_Horizontal_L23mm-W9mm-H9mm-p30mm" V 5880 3300 30  0001 C CNN
+F 2 "pcb:RESIST_35MMX10MM" V 5880 3300 30  0001 C CNN
 F 3 "" H 5950 3300 30  0000 C CNN
 	1    5950 3300
@@
 F 0 "R28" V 6030 3800 50  0000 C CNN
 F 1 "R" V 5950 3800 50  0000 C CNN
-F 2 "Resistors_ThroughHole:Resistor_Ceramic_Horizontal_L23mm-W9mm-H9mm-p30mm" V 5880 3800 30  0001 C CNN
+F 2 "pcb:RESIST_35MMX10MM" V 5880 3800 30  0001 C CNN
 F 3 "" H 5950 3800 30  0000 C CNN
 	1    5950 3800
@@
 F 0 "Q20" H 5550 5300 50  0000 R CNN
 F 1 "MJE350_PNP_EBC" H 5700 5500 50  0000 R CNN
-F 2 "Transistors_TO-220:TO-220_Neutral123_Vertical" H 5450 5350 29  0001 C CNN
+F 2 "pcb:MJE_350_gclass" H 5450 5350 29  0001 C CNN
 F 3 "" H 5250 5250 60  0000 C CNN
 	1    5250 5250
@@
 E
 $Comp
-L CONN_01X03 P6
+L CONN_01X03 P7
 U 1 1 556BD9C4
 P 3850 3150
-F 0 "P6" H 3850 3350 50  0000 C CNN
+F 0 "P7" H 3850 3350 50  0000 C CNN
 F 1 "MJE350" V 3950 3150 50  0000 C CNN
 F 2 "Pin_Headers:Pin_Header_Straight_1x03" H 3850 3150 60  0001 C CNN
@@
 B
 $Comp
-L CONN_01X03 P7
+L CONN_01X03 P8
 U 1 1 556C038A
 P 3850 3850
-F 0 "P7" H 3850 4050 50  0000 C CNN
+F 0 "P8" H 3850 4050 50  0000 C CNN
 F 1 "MJE340" V 3950 3850 50  0000 C CNN
 F 2 "Pin_Headers:Pin_Header_Straight_1x03" H 3850 3850 60  0001 C CNN
@@
 $EndComp
 $Comp
-L CONN_01X03 P9
+L CONN_01X03 P10
 U 1 1 556C0D5A
 P 5550 2750
-F 0 "P9" H 5550 2950 50  0000 C CNN
+F 0 "P10" H 5550 2950 50  0000 C CNN
 F 1 "2SC3281" V 5650 2750 50  0000 C CNN
-F 2 "Pin_Headers:Pin_Header_Straight_1x03" H 5550 2750 60  0001 C CNN
+F 2 "pcb:bornera_grande" H 5550 2750 60  0001 C CNN
 F 3 "" H 5550 2750 60  0000 C CNN
 	1    5550 2750
@@
 $EndComp
 $Comp
-L CONN_01X03 P8
+L CONN_01X03 P9
 U 1 1 556C0DFA
 P 5450 3850
-F 0 "P8" H 5450 4050 50  0000 C CNN
+F 0 "P9" H 5450 4050 50  0000 C CNN
 F 1 "2SA1302" V 5550 3850 50  0000 C CNN
-F 2 "Pin_Headers:Pin_Header_Straight_1x03" H 5450 3850 60  0001 C CNN
+F 2 "pcb:bornera_grande" H 5450 3850 60  0001 C CNN
 F 3 "" H 5450 3850 60  0000 C CNN
 	1    5450 3850
@@
 F 0 "Q14" H 3600 5800 50  0000 R CNN
 F 1 "MPSA06_NPN_EBC" H 3700 5500 50  0000 R CNN
-F 2 "Transistors_TO-220:TO-220_Neutral123_Vertical" H 3500 5850 29  0001 C CNN
+F 2 "pcb:MPSA06-56_TO92_EBC" H 3500 5850 29  0001 C CNN
 F 3 "" H 3300 5750 60  0000 C CNN
 	1    3300 5750
@@
 F 0 "Q16" H 4200 5800 50  0000 R CNN
 F 1 "MPSA06_NPN_EBC" H 4350 5500 50  0000 R CNN
-F 2 "Transistors_TO-220:TO-220_Neutral123_Vertical" H 4100 5850 29  0001 C CNN
+F 2 "pcb:MPSA06-56_TO92_EBC" H 4100 5850 29  0001 C CNN
 F 3 "" H 3900 5750 60  0000 C CNN
 	1    3900 5750
@@
 $EndComp
 $Comp
-L CONN_01X03 P10
+L CONN_01X03 P11
 U 1 1 556C60DA
 P 6300 1950
-F 0 "P10" H 6300 2150 50  0000 C CNN
+F 0 "P11" H 6300 2150 50  0000 C CNN
 F 1 "2SC3281" V 6400 1950 50  0000 C CNN
-F 2 "Pin_Headers:Pin_Header_Straight_1x03" H 6300 1950 60  0001 C CNN
+F 2 "pcb:bornera_grande" H 6300 1950 60  0001 C CNN
 F 3 "" H 6300 1950 60  0000 C CNN
 	1    6300 1950
@@
 E
 $Comp
-L CONN_01X03 P11
+L CONN_01X03 P12
 U 1 1 556C82C3
 P 6300 5050
-F 0 "P11" H 6300 5250 50  0000 C CNN
+F 0 "P12" H 6300 5250 50  0000 C CNN
 F 1 "2SA1302" V 6400 5050 50  0000 C CNN
-F 2 "Pin_Headers:Pin_Header_Straight_1x03" H 6300 5050 60  0001 C CNN
+F 2 "pcb:bornera_grande" H 6300 5050 60  0001 C CNN
 F 3 "" H 6300 5050 60  0000 C CNN
 	1    6300 5050

Commit message: nacho la soba
Parts:
- P7, P8: footprint Pin_Headers:Pin_Header_Straight_1x03 -> pcb:bornera_chica
Changed lines of the file:
@@
 F 0 "P7" H 3850 3350 50  0000 C CNN
 F 1 "MJE350" V 3950 3150 50  0000 C CNN
-F 2 "Pin_Headers:Pin_Header_Straight_1x03" H 3850 3150 60  0001 C CNN
+F 2 "pcb:bornera_chica" H 3850 3150 60  0001 C CNN
 F 3 "" H 3850 3150 60  0000 C CNN
 	1    3850 3150
@@
 F 0 "P8" H 3850 4050 50  0000 C CNN
 F 1 "MJE340" V 3950 3850 50  0000 C CNN
-F 2 "Pin_Headers:Pin_Header_Straight_1x03" H 3850 3850 60  0001 C CNN
+F 2 "pcb:bornera_chica" H 3850 3850 60  0001 C CNN
 F 3 "" H 3850 3850 60  0000 C CNN
 	1    3850 3850
