File: pcb/OPS.sch (KiCad schematic (older format))
At the start: 44 parts, among them P14 MJE350, P15 MJE340, P16 2SA1302, P17 2SC3281, P18 2SC3281, P19 2SA1302, Q13 MPSA56_PNP_EBC, Q14 MPSA06_NPN_EBC, Q15 MPSA56_PNP_EBC, Q16 MPSA06_NPN_EBC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

Commit message: Arreglando PCB
Parts:
- removed Q13: MPSA56_PNP_EBC, pcb:MPSA06-56_TO92_EBC, symbol Q_PNP_EBC
- removed Q14: MPSA06_NPN_EBC, pcb:MPSA06-56_TO92_EBC, symbol Q_NPN_EBC
- added Q13: MPSA06_NPN_EBC, pcb:MPSA06-56_TO92_EBC, symbol Q_NPN_EBC
- added Q14: MPSA56_PNP_EBC, pcb:MPSA06-56_TO92_EBC, symbol Q_PNP_EBC
- added R33, R34: R, Resistors_ThroughHole:Resistor_Horizontal_RM10mm, symbol R
Connections:
- net +VA: now also R33.1
- net -VA: now also Q13.1 (E), R34.1; no longer Q16.1 (E)
- net at Q15.2 (B): now also Q14.1 (E), R33.2; no longer R16.1
- net at D1.1 (K), D3.2 (A): now also Q14.3 (C); no longer Q15.3 (C)
- net at Q16.2 (B), R17.1: now also Q13.3 (C)
- new net: Q14.2 (B), Q15.3 (C), R16.1
- new net: Q13.2 (B), Q16.1 (E), R34.2
Other:
- moved on the sheet: Q15
Changed lines of the file:
@@
 $Descr A4 11693 8268
 encoding utf-8
-Sheet 2 3
+Sheet 2 2
 Title "Amplificador Clase G"
 Date "Mon 01 Jun 2015"
@@
 $EndDescr
 $Comp
-L Q_PNP_EBC Q13
-U 1 1 555E6966
+L Q_PNP_EBC Q15
+U 1 1 555E6967
 P 3300 1350
-F 0 "Q13" H 3600 1400 50  0000 R CNN
-F 1 "MPSA56_PNP_EBC" H 3700 1100 50  0000 R CNN
+F 0 "Q15" H 3600 1400 50  0000 R CNN
+F 1 "MPSA56_PNP_EBC" H 3750 1100 50  0000 R CNN
 F 2 "pcb:MPSA06-56_TO92_EBC" H 3500 1450 29  0001 C CNN
 F 3 "" H 3300 1350 60  0000 C CNN
 	1    3300 1350
 	-1   0    0    1
-$EndComp
-$Comp
-L Q_PNP_EBC Q15
-U 1 1 555E6967
-P 3900 1350
-F 0 "Q15" H 4200 1400 50  0000 R CNN
-F 1 "MPSA56_PNP_EBC" H 4350 1100 50  0000 R CNN
-F 2 "pcb:MPSA06-56_TO92_EBC" H 4100 1450 29  0001 C CNN
-F 3 "" H 3900 1350 60  0000 C CNN
-	1    3900 1350
-	1    0    0    1
 $EndComp
 $Comp
@@
 $EndComp
 $Comp
-L R R17
-U 1 1 555E6978
-P 3200 5200
-F 0 "R17" V 3280 5200 50  0000 C CNN
-F 1 "R" V 3200 5200 50  0000 C CNN
-F 2 "Resistors_ThroughHole:Resistor_Horizontal_RM10mm" V 3130 5200 30  0001 C CNN
-F 3 "" H 3200 5200 30  0000 C CNN
-	1    3200 5200
-	1    0    0    1
-$EndComp
-$Comp
 L D D4
 U 1 1 555E6979
@@
 $Comp
 L GND #PWR038
-U 1 1 555F209B
-P 3200 5050
-F 0 "#PWR038" H 3200 4800 50  0001 C CNN
-F 1 "GND" H 3200 4900 50  0000 C CNN
-F 2 "" H 3200 5050 60  0000 C CNN
-F 3 "" H 3200 5050 60  0000 C CNN
-	1    3200 5050
-	-1   0    0    1
-$EndComp
-$Comp
-L GND #PWR039
 U 1 1 555E698A
 P 3200 2100
-F 0 "#PWR039" H 3200 1850 50  0001 C CNN
+F 0 "#PWR038" H 3200 1850 50  0001 C CNN
 F 1 "GND" H 3200 1950 50  0000 C CNN
 F 2 "" H 3200 2100 60  0000 C CNN
@@
 $EndComp
 $Comp
-L +VA #PWR040
+L +VA #PWR039
 U 1 1 555F2B00
 P 6300 900
-F 0 "#PWR040" H 6300 750 50  0001 C CNN
+F 0 "#PWR039" H 6300 750 50  0001 C CNN
 F 1 "+VA" H 6300 1050 50  0000 C CNN
 F 2 "" H 6300 900 60  0000 C CNN
@@
 $EndComp
 $Comp
-L +VB #PWR041
+L +VB #PWR040
 U 1 1 555F2D0C
 P 6700 2500
-F 0 "#PWR041" H 6700 2350 50  0001 C CNN
+F 0 "#PWR040" H 6700 2350 50  0001 C CNN
 F 1 "+VB" H 6700 2650 50  0000 C CNN
 F 2 "" H 6700 2500 60  0000 C CNN
@@
 $EndComp
 $Comp
-L -VB #PWR042
+L -VB #PWR041
 U 1 1 555F3146
 P 6750 4600
-F 0 "#PWR042" H 6750 4450 50  0001 C CNN
+F 0 "#PWR041" H 6750 4450 50  0001 C CNN
 F 1 "-VB" H 6750 4750 50  0000 C CNN
 F 2 "" H 6750 4600 60  0000 C CNN
@@
 $EndComp
 $Comp
-L -VA #PWR043
+L -VA #PWR042
 U 1 1 555F3328
 P 6300 6200
-F 0 "#PWR043" H 6300 6050 50  0001 C CNN
+F 0 "#PWR042" H 6300 6050 50  0001 C CNN
 F 1 "-VA" H 6300 6350 50  0000 C CNN
 F 2 "" H 6300 6200 60  0000 C CNN
@@
 Acoplación\nTérmica\n
 $Comp
-L Q_NPN_EBC Q14
-U 1 1 556C4C7C
-P 3300 5750
-F 0 "Q14" H 3600 5800 50  0000 R CNN
-F 1 "MPSA06_NPN_EBC" H 3700 5500 50  0000 R CNN
-F 2 "pcb:MPSA06-56_TO92_EBC" H 3500 5850 29  0001 C CNN
-F 3 "" H 3300 5750 60  0000 C CNN
-	1    3300 5750
-	-1   0    0    -1
-$EndComp
-$Comp
-L Q_NPN_EBC Q16
-U 1 1 556C5042
-P 3900 5750
-F 0 "Q16" H 4200 5800 50  0000 R CNN
-F 1 "MPSA06_NPN_EBC" H 4350 5500 50  0000 R CNN
-F 2 "pcb:MPSA06-56_TO92_EBC" H 4100 5850 29  0001 C CNN
-F 3 "" H 3900 5750 60  0000 C CNN
-	1    3900 5750
-	1    0    0    -1
-$EndComp
-$Comp
 L CONN_01X03 P18
 U 1 1 556C60DA
@@
 $EndComp
 $Comp
-L GND #PWR044
+L GND #PWR043
 U 1 1 556CC8CC
 P 5750 5750
-F 0 "#PWR044" H 5750 5500 50  0001 C CNN
+F 0 "#PWR043" H 5750 5500 50  0001 C CNN
 F 1 "GND" H 5750 5600 50  0000 C CNN
 F 2 "" H 5750 5750 60  0000 C CNN
@@
 $EndComp
 $Comp
-L GND #PWR045
+L GND #PWR044
 U 1 1 556CCB94
 P 6150 1300
-F 0 "#PWR045" H 6150 1050 50  0001 C CNN
+F 0 "#PWR044" H 6150 1050 50  0001 C CNN
 F 1 "GND" H 6150 1150 50  0000 C CNN
 F 2 "" H 6150 1300 60  0000 C CNN
@@
 $EndComp
 $Comp
-L GND #PWR046
+L GND #PWR045
 U 1 1 556CECB0
 P 6600 5000
-F 0 "#PWR046" H 6600 4750 50  0001 C CNN
+F 0 "#PWR045" H 6600 4750 50  0001 C CNN
 F 1 "GND" H 6600 4850 50  0000 C CNN
 F 2 "" H 6600 5000 60  0000 C CNN
@@
 $EndComp
 $Comp
-L GND #PWR047
+L GND #PWR046
 U 1 1 556CF118
 P 6600 2200
-F 0 "#PWR047" H 6600 1950 50  0001 C CNN
+F 0 "#PWR046" H 6600 1950 50  0001 C CNN
 F 1 "GND" H 6600 2050 50  0000 C CNN
 F 2 "" H 6600 2200 60  0000 C CNN
@@
 OUT
 $Comp
-L GND #PWR048
+L GND #PWR047
 U 1 1 556E0BD9
 P 7200 4250
-F 0 "#PWR048" H 7200 4000 50  0001 C CNN
+F 0 "#PWR047" H 7200 4000 50  0001 C CNN
 F 1 "GND" H 7200 4100 50  0000 C CNN
 F 2 "" H 7200 4250 60  0000 C CNN
@@
 Connection ~ 6150 900
 Wire Wire Line
-	6150 950  6150 900
+	6150 900  6150 950
 Connection ~ 6800 3550
 Wire Wire Line
@@
 Wire Wire Line
 	4450 3000 4450 3100
-Wire Wire Line
-	4000 1550 4000 2050
 Wire Notes Line
 	3450 2650 3450 4500
@@
 Connection ~ 6000 6200
 Wire Wire Line
-	6000 5050 6000 6200
-Wire Wire Line
-	6100 5050 6000 5050
+	6000 6200 6000 5050
+Wire Wire Line
+	6000 5050 6100 5050
 Wire Wire Line
 	5950 5150 6100 5150
@@
 Connection ~ 4950 4150
 Wire Wire Line
-	4950 4350 4950 4000
+	4950 4000 4950 4350
 Connection ~ 4950 6200
 Wire Wire Line
-	4950 4750 4950 6200
+	4950 6200 4950 4750
 Connection ~ 5350 6200
 Wire Wire Line
@@
 	4700 5250 5050 5250
 Wire Wire Line
-	4400 5250 4000 5250
-Wire Wire Line
 	4450 4550 4650 4550
 Connection ~ 4000 4550
 Wire Wire Line
-	4150 4550 4000 4550
-Connection ~ 4000 5250
-Wire Wire Line
-	4000 5550 4000 4900
+	4000 4550 4150 4550
 Connection ~ 4000 4400
 Wire Wire Line
@@
 Wire Wire Line
 	3650 4400 4450 4400
-Connection ~ 4000 6200
-Wire Wire Line
-	4000 6200 4000 5950
-Wire Wire Line
-	3200 6200 6300 6200
-Wire Wire Line
-	3200 5950 3200 6200
-Wire Wire Line
-	3500 5750 3700 5750
-Wire Wire Line
-	3500 5550 3500 5750
-Wire Wire Line
-	3200 5550 3500 5550
-Wire Wire Line
-	3200 5550 3200 5350
 Wire Wire Line
 	5950 3450 5950 3650
@@
 Connection ~ 4950 900
 Wire Wire Line
-	4950 2350 4950 900
+	4950 900  4950 2350
 Connection ~ 5950 900
 Connection ~ 5350 900
@@
 Connection ~ 4000 900
 Wire Wire Line
-	4000 900  4000 1150
-Wire Wire Line
 	3200 900  6300 900
 Wire Wire Line
 	3200 1150 3200 900
 Wire Wire Line
-	3500 1350 3700 1350
-Wire Wire Line
-	3500 1550 3500 1350
-Wire Wire Line
-	3200 1550 3500 1550
+	3500 1350 4000 1350
+Wire Wire Line
+	4750 3400 4750 2950
+Wire Wire Line
+	4750 3700 4750 4150
+Wire Wire Line
+	4950 3700 4950 3400
+Wire Wire Line
+	7200 4200 7200 4250
+$Comp
+L R R33
+U 1 1 5587C061
+P 4000 1150
+F 0 "R33" V 4080 1150 50  0000 C CNN
+F 1 "R" V 4000 1150 50  0000 C CNN
+F 2 "Resistors_ThroughHole:Resistor_Horizontal_RM10mm" V 3930 1150 30  0001 C CNN
+F 3 "" H 4000 1150 30  0000 C CNN
+	1    4000 1150
+	1    0    0    -1
+$EndComp
+Wire Wire Line
+	4000 900  4000 1000
+$Comp
+L Q_PNP_EBC Q14
+U 1 1 5587C528
+P 3900 1600
+F 0 "Q14" H 4200 1650 50  0000 R CNN
+F 1 "MPSA56_PNP_EBC" H 4350 1350 50  0000 R CNN
+F 2 "pcb:MPSA06-56_TO92_EBC" H 4100 1700 29  0001 C CNN
+F 3 "" H 3900 1600 60  0000 C CNN
+	1    3900 1600
+	1    0    0    1
+$EndComp
+Wire Wire Line
+	4000 1300 4000 1400
+Connection ~ 4000 1350
+Wire Wire Line
+	3700 1600 3200 1600
 Wire Wire Line
 	3200 1550 3200 1750
-Wire Wire Line
-	4750 3400 4750 2950
-Wire Wire Line
-	4750 3700 4750 4150
-Wire Wire Line
-	4950 3700 4950 3400
-Wire Wire Line
-	7200 4200 7200 4250
-$Sheet
-S 9550 3650 500  150
-U 5578D376
-F0 "Sheet5578D375" 60
-F1 "file5578D375.sch" 60
-$EndSheet
+Connection ~ 3200 1600
+Wire Wire Line
+	4000 1800 4000 2050
+$Comp
+L R R17
+U 1 1 5587DC07
+P 3200 5200
+F 0 "R17" V 3280 5200 50  0000 C CNN
+F 1 "R" V 3200 5200 50  0000 C CNN
+F 2 "Resistors_ThroughHole:Resistor_Horizontal_RM10mm" V 3130 5200 30  0001 C CNN
+F 3 "" H 3200 5200 30  0000 C CNN
+	1    3200 5200
+	1    0    0    1
+$EndComp
+$Comp
+L GND #PWR048
+U 1 1 5587DC0D
+P 3200 5000
+F 0 "#PWR048" H 3200 4750 50  0001 C CNN
+F 1 "GND" H 3200 4850 50  0000 C CNN
+F 2 "" H 3200 5000 60  0000 C CNN
+F 3 "" H 3200 5000 60  0000 C CNN
+	1    3200 5000
+	1    0    0    1
+$EndComp
+Wire Wire Line
+	3200 5000 3200 5050
+Connection ~ 4000 6200
+Wire Wire Line
+	3200 5950 3200 6200
+Wire Wire Line
+	3500 5750 4000 5750
+$Comp
+L R R34
+U 1 1 5587DC20
+P 4000 5950
+F 0 "R34" V 4080 5950 50  0000 C CNN
+F 1 "R" V 4000 5950 50  0000 C CNN
+F 2 "Resistors_ThroughHole:Resistor_Horizontal_RM10mm" V 3930 5950 30  0001 C CNN
+F 3 "" H 4000 5950 30  0000 C CNN
+	1    4000 5950
+	1    0    0    1
+$EndComp
+Wire Wire Line
+	4000 6200 4000 6100
+Wire Wire Line
+	4000 5800 4000 5700
+Connection ~ 4000 5750
+Wire Wire Line
+	3700 5500 3200 5500
+Wire Wire Line
+	3200 5550 3200 5350
+Connection ~ 3200 5500
+Wire Wire Line
+	4000 4900 4000 5300
+Wire Wire Line
+	3200 6200 5350 6200
+$Comp
+L Q_NPN_EBC Q13
+U 1 1 5587E793
+P 3300 5750
+F 0 "Q13" H 3600 5800 50  0000 R CNN
+F 1 "MPSA06_NPN_EBC" H 3700 5500 50  0000 R CNN
+F 2 "pcb:MPSA06-56_TO92_EBC" H 3500 5850 29  0001 C CNN
+F 3 "" H 3300 5750 60  0000 C CNN
+	1    3300 5750
+	-1   0    0    -1
+$EndComp
+$Comp
+L Q_NPN_EBC Q16
+U 1 1 5587E835
+P 3900 5500
+F 0 "Q16" H 4200 5550 50  0000 R CNN
+F 1 "MPSA06_NPN_EBC" H 4350 5250 50  0000 R CNN
+F 2 "pcb:MPSA06-56_TO92_EBC" H 4100 5600 29  0001 C CNN
+F 3 "" H 3900 5500 60  0000 C CNN
+	1    3900 5500
+	1    0    0    -1
+$EndComp
+Wire Wire Line
+	4400 5250 4000 5250
+Connection ~ 4000 5250
+Wire Wire Line
+	5300 6200 6300 6200
 $EndSCHEMATC
