File: pcb/amplificador_gclass.sch (KiCad schematic (older format))
At the start: 36 parts, among them P1 CONN_01X02, P2 CONN_01X02, P3 CONN_01X02, P4 CONN_01X02, P5 BNC, P6 BNC, Q1 Q_PNP_EBC, Q10 Q_NPN_EBC, Q11 Q_PNP_EBC, Q12 Q_NPN_EBC, Q2 Q_PNP_EBC, Q3 Q_NPN_EBC, Q4 Q_PNP_EBC, Q5 Q_NPN_EBC, Q6 Q_PNP_EBC, Q7 Q_PNP_EBC, Q8 Q_PNP_EBC, Q9 Q_PNP_EBC

Commit message: Sigo con el fucking error de power conectors...
Connections:
- net labels added: GND_
- wire segments 60 -> 62
Changed lines of the file:
@@
-$EndComp
-$Comp
-L GND #PWR01
-U 1 1 555E73FE
-P 2250 4600
-F 0 "#PWR01" H 2250 4350 50  0001 C CNN
-F 1 "GND" H 2250 4450 50  0000 C CNN
-F 2 "" H 2250 4600 60  0000 C CNN
-F 3 "" H 2250 4600 60  0000 C CNN
-	1    2250 4600
-	1    0    0    -1
-$EndComp
-$Comp
-L GND #PWR02
-U 1 1 555E752F
-P 6500 5450
-F 0 "#PWR02" H 6500 5200 50  0001 C CNN
-F 1 "GND" H 6500 5300 50  0000 C CNN
-F 2 "" H 6500 5450 60  0000 C CNN
-F 3 "" H 6500 5450 60  0000 C CNN
-	1    6500 5450
-	1    0    0    -1
 $EndComp
 $Comp
@@
 F 3 "" H 5200 2450 30  0000 C CNN
 	1    5200 2450
-	1    0    0    -1
-$EndComp
-$Comp
-L GND #PWR03
-U 1 1 555E8B8F
-P 5200 2700
-F 0 "#PWR03" H 5200 2450 50  0001 C CNN
-F 1 "GND" H 5200 2550 50  0000 C CNN
-F 2 "" H 5200 2700 60  0000 C CNN
-F 3 "" H 5200 2700 60  0000 C CNN
-	1    5200 2700
 	1    0    0    -1
 $EndComp
@@
 	0    1    1    0
 $EndComp
-Text GLabel 8500 5900 2    60   Input ~ 0
--VA
 Text GLabel 8650 3850 2    60   Input ~ 0
 TO_OPS
-Text GLabel 8600 1500 2    60   Input ~ 0
-+VA
 Text Notes 8750 3700 0    60   ~ 0
 To Output Stage\n
@@
 $EndComp
 $Comp
-L GND #PWR04
-U 1 1 555E8C11
-P 1900 4550
-F 0 "#PWR04" H 1900 4300 50  0001 C CNN
-F 1 "GND" H 1900 4400 50  0000 C CNN
-F 2 "" H 1900 4550 60  0000 C CNN
-F 3 "" H 1900 4550 60  0000 C CNN
-	1    1900 4550
-	1    0    0    -1
-$EndComp
-$Comp
 L BNC P5
 U 1 1 555E9171
@@
 OUT
 $Comp
-L GND #PWR05
+L GND #PWR01
 U 1 1 555E93F0
 P 1900 3350
-F 0 "#PWR05" H 1900 3100 50  0001 C CNN
+F 0 "#PWR01" H 1900 3100 50  0001 C CNN
 F 1 "GND" H 1900 3200 50  0000 C CNN
 F 2 "" H 1900 3350 60  0000 C CNN
@@
 	0    -1   -1   0
 $EndComp
-Text GLabel 800  3700 3    60   Input ~ 0
-+VB
-Text GLabel 1350 3700 3    60   Input ~ 0
--VB
-Text GLabel 1350 2800 3    60   Input ~ 0
--VA
-Text GLabel 800  2800 3    60   Input ~ 0
-+VA
 $Comp
 L CONN_01X02 P1
@@
 $EndComp
 $Comp
-L GND #PWR06
+L GND #PWR02
 U 1 1 555EA3AF
 P 900 3700
-F 0 "#PWR06" H 900 3450 50  0001 C CNN
+F 0 "#PWR02" H 900 3450 50  0001 C CNN
 F 1 "GND" H 900 3550 50  0000 C CNN
 F 2 "" H 900 3700 60  0000 C CNN
@@
 $EndComp
 $Comp
-L GND #PWR07
+L GND #PWR03
 U 1 1 555EA426
 P 900 2800
-F 0 "#PWR07" H 900 2550 50  0001 C CNN
+F 0 "#PWR03" H 900 2550 50  0001 C CNN
 F 1 "GND" H 900 2650 50  0000 C CNN
 F 2 "" H 900 2800 60  0000 C CNN
@@
 $EndComp
 $Comp
-L GND #PWR08
+L GND #PWR04
 U 1 1 555EA479
 P 1450 2800
-F 0 "#PWR08" H 1450 2550 50  0001 C CNN
+F 0 "#PWR04" H 1450 2550 50  0001 C CNN
 F 1 "GND" H 1450 2650 50  0000 C CNN
 F 2 "" H 1450 2800 60  0000 C CNN
@@
 $EndComp
 $Comp
-L GND #PWR09
+L GND #PWR05
 U 1 1 555EA4CC
 P 1450 3700
-F 0 "#PWR09" H 1450 3450 50  0001 C CNN
+F 0 "#PWR05" H 1450 3450 50  0001 C CNN
 F 1 "GND" H 1450 3550 50  0000 C CNN
 F 2 "" H 1450 3700 60  0000 C CNN
@@
 	2650 4550 2650 4750
 Wire Wire Line
-	1900 4350 1900 4550
-Wire Wire Line
-	2250 4600 2250 4550
+	1900 4350 1900 5050
+Wire Wire Line
+	2250 4550 2250 5050
 Wire Wire Line
 	2650 4150 3450 4150
@@
 Wire Wire Line
 	5200 2700 5200 2600
-$Comp
-L GND #PWR010
+Wire Wire Line
+	7550 2700 7550 2600
+$Comp
+L GND #PWR06
 U 1 1 555EFF7C
 P 2650 5050
-F 0 "#PWR010" H 2650 4800 50  0001 C CNN
+F 0 "#PWR06" H 2650 4800 50  0001 C CNN
 F 1 "GND" H 2650 4900 50  0000 C CNN
 F 2 "" H 2650 5050 60  0000 C CNN
@@
 	1    0    0    -1
 $EndComp
-$Comp
-L GND #PWR011
-U 1 1 555F056C
-P 7800 4300
-F 0 "#PWR011" H 7800 4050 50  0001 C CNN
-F 1 "GND" H 7800 4150 50  0000 C CNN
-F 2 "" H 7800 4300 60  0000 C CNN
-F 3 "" H 7800 4300 60  0000 C CNN
-	1    7800 4300
+Wire Wire Line
+	7800 4200 7800 4300
+Wire Wire Line
+	1900 5050 2650 5050
+Connection ~ 2250 5050
+$Comp
+L +VA #PWR07
+U 1 1 555F1574
+P 8600 1500
+F 0 "#PWR07" H 8600 1350 50  0001 C CNN
+F 1 "+VA" H 8600 1650 50  0000 C CNN
+F 2 "" H 8600 1500 60  0000 C CNN
+F 3 "" H 8600 1500 60  0000 C CNN
+	1    8600 1500
+	0    1    1    0
+$EndComp
+$Comp
+L -VA #PWR08
+U 1 1 555F1C4D
+P 8500 5900
+F 0 "#PWR08" H 8500 5750 50  0001 C CNN
+F 1 "-VA" H 8500 6050 50  0000 C CNN
+F 2 "" H 8500 5900 60  0000 C CNN
+F 3 "" H 8500 5900 60  0000 C CNN
+	1    8500 5900
+	0    1    1    0
+$EndComp
+$Comp
+L GND #PWR09
+U 1 1 555F1F71
+P 5200 2700
+F 0 "#PWR09" H 5200 2450 50  0001 C CNN
+F 1 "GND" H 5200 2550 50  0000 C CNN
+F 2 "" H 5200 2700 60  0000 C CNN
+F 3 "" H 5200 2700 60  0000 C CNN
+	1    5200 2700
+	1    0    0    -1
+$EndComp
+$Comp
+L +VA #PWR010
+U 1 1 555F36E5
+P 800 2800
+F 0 "#PWR010" H 800 2650 50  0001 C CNN
+F 1 "+VA" H 800 2950 50  0000 C CNN
+F 2 "" H 800 2800 60  0000 C CNN
+F 3 "" H 800 2800 60  0000 C CNN
+	1    800  2800
 	-1   0    0    1
 $EndComp
 $Comp
-L GND #PWR012
-U 1 1 555EA46B
+L +VB #PWR011
+U 1 1 555F3741
+P 800 3700
+F 0 "#PWR011" H 800 3550 50  0001 C CNN
+F 1 "+VB" H 800 3850 50  0000 C CNN
+F 2 "" H 800 3700 60  0000 C CNN
+F 3 "" H 800 3700 60  0000 C CNN
+	1    800  3700
+	-1   0    0    1
+$EndComp
+$Comp
+L -VA #PWR012
+U 1 1 555F379D
+P 1350 2800
+F 0 "#PWR012" H 1350 2650 50  0001 C CNN
+F 1 "-VA" H 1350 2950 50  0000 C CNN
+F 2 "" H 1350 2800 60  0000 C CNN
+F 3 "" H 1350 2800 60  0000 C CNN
+	1    1350 2800
+	-1   0    0    1
+$EndComp
+$Comp
+L -VB #PWR013
+U 1 1 555F37F9
+P 1350 3700
+F 0 "#PWR013" H 1350 3550 50  0001 C CNN
+F 1 "-VB" H 1350 3850 50  0000 C CNN
+F 2 "" H 1350 3700 60  0000 C CNN
+F 3 "" H 1350 3700 60  0000 C CNN
+	1    1350 3700
+	-1   0    0    1
+$EndComp
+$Comp
+L GND_ #PWR014
+U 1 1 555FB72E
+P 6500 5450
+F 0 "#PWR014" H 6500 5200 50  0001 C CNN
+F 1 "GND_" H 6500 5300 50  0000 C CNN
+F 2 "" H 6500 5450 60  0000 C CNN
+F 3 "" H 6500 5450 60  0000 C CNN
+	1    6500 5450
+	1    0    0    -1
+$EndComp
+$Comp
+L GND_ #PWR015
+U 1 1 555FB944
+P 7800 4200
+F 0 "#PWR015" H 7800 3950 50  0001 C CNN
+F 1 "GND_" H 7800 4050 50  0000 C CNN
+F 2 "" H 7800 4200 60  0000 C CNN
+F 3 "" H 7800 4200 60  0000 C CNN
+	1    7800 4200
+	-1   0    0    1
+$EndComp
+$Comp
+L GND_ #PWR016
+U 1 1 555FBF2F
 P 7550 2700
-F 0 "#PWR012" H 7550 2450 50  0001 C CNN
-F 1 "GND" H 7550 2550 50  0000 C CNN
+F 0 "#PWR016" H 7550 2450 50  0001 C CNN
+F 1 "GND_" H 7550 2550 50  0000 C CNN
 F 2 "" H 7550 2700 60  0000 C CNN
 F 3 "" H 7550 2700 60  0000 C CNN
 	1    7550 2700
-	-1   0    0    -1
-$EndComp
-Wire Wire Line
-	7550 2700 7550 2600
+	1    0    0    -1
+$EndComp
 $EndSCHEMATC

Commit message: Problema sobre power conections arreglado, ahora hay otros quilombos, creo que tiene que ver con el encapsulado de los transistores.
Parts:
- removed P6: BNC, Sockets_BNC:BNC_Socket_TYCO-AMP, symbol BNC
- added P5: BNC, Sockets_BNC:BNC_Socket_TYCO-AMP, symbol BNC
- C1, C2, C3, C4: footprint Capacitors_SMD:C_0201 -> Capacitors_SMD:C_0603_HandSoldering
- Q1, Q10, Q11, Q12, Q2, Q3, Q4, Q5, Q6, Q7, Q8, Q9: footprint Transistors_TO-220:TO-220_Bipolar-BCE_Horizontal -> Transistors_TO-220:TO-220_Bipolar-BCE_Vertical_LargePads
- R1, R10, R11, R12, R13, R14, R2, R3, R4, R5, R6, R7, R8, R9: footprint Resistors_SMD:R_0201 -> Resistors_SMD:R_0603_HandSoldering
- renumbered P5 to P6
Connections:
- net labels added: IN
- net labels removed: GND_
- wire segments 62 -> 66
Other:
- moved on the sheet: P1, P2, P3, P4, P6

Commit message: Sigo trabajando en el PCB usando Kicad, necesito mas info sobre los diodos para continuar.
Parts:
- Q1, Q11, Q2, Q4, Q6, Q7, Q8, Q9: value Q_PNP_EBC -> MPSA56_PNP_EBC
- Q10, Q12, Q3, Q5: value Q_NPN_EBC -> MPSA06_NPN_EBC
Changed lines of the file:
@@
 $EndDescr
-$Comp
-L Q_PNP_EBC Q1
-U 1 1 555E57F7
-P 2950 4150
-F 0 "Q1" H 3250 4200 50  0000 R CNN
-F 1 "Q_PNP_EBC" H 3550 4100 50  0000 R CNN
-F 2 "Transistors_TO-220:TO-220_Bipolar-BCE_Vertical_LargePads" H 3150 4250 29  0001 C CNN
-F 3 "" H 2950 4150 60  0000 C CNN
-	1    2950 4150
-	1    0    0    1
-$EndComp
-$Comp
-L Q_PNP_EBC Q2
-U 1 1 555E586E
-P 3650 4150
-F 0 "Q2" H 3950 4200 50  0000 R CNN
-F 1 "Q_PNP_EBC" H 4250 4100 50  0000 R CNN
-F 2 "Transistors_TO-220:TO-220_Bipolar-BCE_Vertical_LargePads" H 3850 4250 29  0001 C CNN
-F 3 "" H 3650 4150 60  0000 C CNN
-	1    3650 4150
-	1    0    0    1
-$EndComp
-$Comp
-L Q_PNP_EBC Q7
-U 1 1 555E58EC
-P 5200 4150
-F 0 "Q7" H 5500 4200 50  0000 R CNN
-F 1 "Q_PNP_EBC" H 5800 4100 50  0000 R CNN
-F 2 "Transistors_TO-220:TO-220_Bipolar-BCE_Vertical_LargePads" H 5400 4250 29  0001 C CNN
-F 3 "" H 5200 4150 60  0000 C CNN
-	1    5200 4150
-	-1   0    0    1
-$EndComp
-$Comp
-L Q_PNP_EBC Q8
-U 1 1 555E597A
-P 5900 4150
-F 0 "Q8" H 6200 4200 50  0000 R CNN
-F 1 "Q_PNP_EBC" H 6500 4100 50  0000 R CNN
-F 2 "Transistors_TO-220:TO-220_Bipolar-BCE_Vertical_LargePads" H 6100 4250 29  0001 C CNN
-F 3 "" H 5900 4150 60  0000 C CNN
-	1    5900 4150
-	-1   0    0    1
-$EndComp
-$Comp
-L Q_PNP_EBC Q4
-U 1 1 555E5D61
-P 4450 1900
-F 0 "Q4" H 4750 1950 50  0000 R CNN
-F 1 "Q_PNP_EBC" H 5050 1850 50  0000 R CNN
-F 2 "Transistors_TO-220:TO-220_Bipolar-BCE_Vertical_LargePads" H 4650 2000 29  0001 C CNN
-F 3 "" H 4450 1900 60  0000 C CNN
-	1    4450 1900
-	-1   0    0    1
-$EndComp
 $Comp
 L Q_PNP_EBC Q6
@@
 P 5100 1900
 F 0 "Q6" H 5400 1950 50  0000 R CNN
-F 1 "Q_PNP_EBC" H 5700 1850 50  0000 R CNN
+F 1 "MPSA56_PNP_EBC" H 5700 1850 50  0000 R CNN
 F 2 "Transistors_TO-220:TO-220_Bipolar-BCE_Vertical_LargePads" H 5300 2000 29  0001 C CNN
 F 3 "" H 5100 1900 60  0000 C CNN
@@
 P 3850 4950
 F 0 "Q3" H 4150 5000 50  0000 R CNN
-F 1 "Q_NPN_EBC" H 4450 4900 50  0000 R CNN
+F 1 "MPSA06_NPN_EBC" H 4450 4900 50  0000 R CNN
 F 2 "Transistors_TO-220:TO-220_Bipolar-BCE_Vertical_LargePads" H 4050 5050 29  0001 C CNN
 F 3 "" H 3850 4950 60  0000 C CNN
@@
 P 5000 4950
 F 0 "Q5" H 5300 5000 50  0000 R CNN
-F 1 "Q_NPN_EBC" H 5600 4900 50  0000 R CNN
+F 1 "MPSA06_NPN_EBC" H 5600 4900 50  0000 R CNN
 F 2 "Transistors_TO-220:TO-220_Bipolar-BCE_Vertical_LargePads" H 5200 5050 29  0001 C CNN
 F 3 "" H 5000 4950 60  0000 C CNN
@@
 OUT
 $Comp
-L Q_PNP_EBC Q11
-U 1 1 555EA459
-P 8300 1900
-F 0 "Q11" H 8600 1950 50  0000 R CNN
-F 1 "Q_PNP_EBC" H 8900 1850 50  0000 R CNN
-F 2 "Transistors_TO-220:TO-220_Bipolar-BCE_Vertical_LargePads" H 8500 2000 29  0001 C CNN
-F 3 "" H 8300 1900 60  0000 C CNN
-	1    8300 1900
-	1    0    0    1
-$EndComp
-$Comp
 L Q_PNP_EBC Q9
 U 1 1 555EA45F
 P 7650 1900
 F 0 "Q9" H 7950 1950 50  0000 R CNN
-F 1 "Q_PNP_EBC" H 8250 1850 50  0000 R CNN
+F 1 "MPSA56_PNP_EBC" H 8250 1850 50  0000 R CNN
 F 2 "Transistors_TO-220:TO-220_Bipolar-BCE_Vertical_LargePads" H 7850 2000 29  0001 C CNN
 F 3 "" H 7650 1900 60  0000 C CNN
@@
 	1    7550 2450
 	-1   0    0    -1
-$EndComp
-$Comp
-L Q_NPN_EBC Q10
-U 1 1 555EA80B
-P 7700 4500
-F 0 "Q10" H 8000 4550 50  0000 R CNN
-F 1 "Q_NPN_EBC" H 8300 4450 50  0000 R CNN
-F 2 "Transistors_TO-220:TO-220_Bipolar-BCE_Vertical_LargePads" H 7900 4600 29  0001 C CNN
-F 3 "" H 7700 4500 60  0000 C CNN
-	1    7700 4500
-	1    0    0    -1
-$EndComp
-$Comp
-L Q_NPN_EBC Q12
-U 1 1 555EA8E5
-P 8300 4150
-F 0 "Q12" H 8600 4200 50  0000 R CNN
-F 1 "Q_NPN_EBC" H 8900 4100 50  0000 R CNN
-F 2 "Transistors_TO-220:TO-220_Bipolar-BCE_Vertical_LargePads" H 8500 4250 29  0001 C CNN
-F 3 "" H 8300 4150 60  0000 C CNN
-	1    8300 4150
-	1    0    0    -1
 $EndComp
 $Comp
@@
 Wire Notes Line
 	1050 3700 1050 2100
+$Comp
+L Q_PNP_EBC Q4
+U 1 1 556D7105
+P 4450 1900
+F 0 "Q4" H 4750 1950 50  0000 R CNN
+F 1 "MPSA56_PNP_EBC" H 5050 1850 50  0000 R CNN
+F 2 "Transistors_TO-220:TO-220_Bipolar-BCE_Vertical_LargePads" H 4650 2000 29  0001 C CNN
+F 3 "" H 4450 1900 60  0000 C CNN
+	1    4450 1900
+	-1   0    0    1
+$EndComp
+$Comp
+L Q_PNP_EBC Q7
+U 1 1 556D735C
+P 5200 4150
+F 0 "Q7" H 5500 4200 50  0000 R CNN
+F 1 "MPSA56_PNP_EBC" H 5800 4100 50  0000 R CNN
+F 2 "Transistors_TO-220:TO-220_Bipolar-BCE_Vertical_LargePads" H 5400 4250 29  0001 C CNN
+F 3 "" H 5200 4150 60  0000 C CNN
+	1    5200 4150
+	-1   0    0    1
+$EndComp
+$Comp
+L Q_PNP_EBC Q8
+U 1 1 556D7418
+P 5900 4150
+F 0 "Q8" H 6200 4200 50  0000 R CNN
+F 1 "MPSA56_PNP_EBC" H 6500 4100 50  0000 R CNN
+F 2 "Transistors_TO-220:TO-220_Bipolar-BCE_Vertical_LargePads" H 6100 4250 29  0001 C CNN
+F 3 "" H 5900 4150 60  0000 C CNN
+	1    5900 4150
+	-1   0    0    1
+$EndComp
+$Comp
+L Q_PNP_EBC Q2
+U 1 1 556D7A6B
+P 3650 4150
+F 0 "Q2" H 3950 4200 50  0000 R CNN
+F 1 "MPSA56_PNP_EBC" H 4250 4100 50  0000 R CNN
+F 2 "Transistors_TO-220:TO-220_Bipolar-BCE_Vertical_LargePads" H 3850 4250 29  0001 C CNN
+F 3 "" H 3650 4150 60  0000 C CNN
+	1    3650 4150
+	1    0    0    1
+$EndComp
+$Comp
+L Q_PNP_EBC Q1
+U 1 1 556D7B31
+P 2950 4150
+F 0 "Q1" H 3250 4200 50  0000 R CNN
+F 1 "MPSA56_PNP_EBC" H 3550 4100 50  0000 R CNN
+F 2 "Transistors_TO-220:TO-220_Bipolar-BCE_Vertical_LargePads" H 3150 4250 29  0001 C CNN
+F 3 "" H 2950 4150 60  0000 C CNN
+	1    2950 4150
+	1    0    0    1
+$EndComp
+$Comp
+L Q_PNP_EBC Q11
+U 1 1 556D7C97
+P 8300 1900
+F 0 "Q11" H 8600 1950 50  0000 R CNN
+F 1 "MPSA56_PNP_EBC" H 8900 1850 50  0000 R CNN
+F 2 "Transistors_TO-220:TO-220_Bipolar-BCE_Vertical_LargePads" H 8500 2000 29  0001 C CNN
+F 3 "" H 8300 1900 60  0000 C CNN
+	1    8300 1900
+	1    0    0    1
+$EndComp
+$Comp
+L Q_NPN_EBC Q10
+U 1 1 556D81CA
+P 7700 4500
+F 0 "Q10" H 8000 4550 50  0000 R CNN
+F 1 "MPSA06_NPN_EBC" H 8300 4450 50  0000 R CNN
+F 2 "Transistors_TO-220:TO-220_Bipolar-BCE_Vertical_LargePads" H 7900 4600 29  0001 C CNN
+F 3 "" H 7700 4500 60  0000 C CNN
+	1    7700 4500
+	1    0    0    -1
+$EndComp
+$Comp
+L Q_NPN_EBC Q12
+U 1 1 556D8298
+P 8300 4150
+F 0 "Q12" H 8600 4200 50  0000 R CNN
+F 1 "MPSA06_NPN_EBC" H 8900 4100 50  0000 R CNN
+F 2 "Transistors_TO-220:TO-220_Bipolar-BCE_Vertical_LargePads" H 8500 4250 29  0001 C CNN
+F 3 "" H 8300 4150 60  0000 C CNN
+	1    8300 4150
+	1    0    0    -1
+$EndComp
 $EndSCHEMATC

Commit message: Agrego algunos datasheets, el export kicad en pdf y sigo trabajando en el PCB
Parts:
- removed P5, P6: BNC, Sockets_BNC:BNC_Socket_TYCO-AMP, symbol BNC
- removed R14: R, Resistors_SMD:R_0603_HandSoldering, symbol R
- added C3, C6: C, Capacitors_Elko_ThroughHole:Elko_vert_11.5x8mm_RM3.5, symbol C
- added C4, C5: C, Capacitors_Elko_ThroughHole:Elko_vert_11.2x6.3mm_RM2.5_CopperClear, symbol C
- added CON1: AUDIO_IN, symbol BARREL_JACK
- added JP1: JUMPER, Socket_Strips:Socket_Strip_Angled_1x02, symbol JUMPER
- added P5: OUT, symbol CONN_01X02
- added R10, R15: R, Resistors_SMD:R_0603_HandSoldering, symbol R
- added RV1: POT, symbol POT
- C1: footprint Capacitors_SMD:C_0603_HandSoldering -> Capacitors_Elko_ThroughHole:Elko_vert_11.2x6.3mm_RM2.5_CopperClear
- C2: footprint Capacitors_SMD:C_0603_HandSoldering -> Capacitors_Elko_ThroughHole:Elko_vert_11.5x8mm_RM3.5
- C7: renamed from C3; footprint Capacitors_SMD:C_0603_HandSoldering -> Capacitors_Elko_ThroughHole:Elko_vert_11.5x8mm_RM3.5
- C8: renamed from C4; footprint Capacitors_SMD:C_0603_HandSoldering -> Capacitors_Elko_ThroughHole:Elko_vert_11.5x8mm_RM3.5
- P1: value CONN_01X02 -> +VA_GND
- P2: value CONN_01X02 -> +VB_GND
- P3: value CONN_01X02 -> -VA_GND
- P4: value CONN_01X02 -> -VB_GND
- Q1, Q10, Q11, Q12, Q2, Q3, Q4, Q5, Q6, Q7, Q8, Q9: footprint Transistors_TO-220:TO-220_Bipolar-BCE_Vertical_LargePads -> Transistors_TO-220:TO-220_Neutral123_Vertical
- renumbered R10 to R11, R11 to R12, R12 to R13, R13 to R14
Connections:
- net -VA: no longer R14.2, R5.2, R8.2
- net GND: now also R14.2, C4.2, CON1.2, CON1.3, P5.1 (P1), R10.1, R15.2
- net IN: now also CON1.1
- net OUT: now also P5.2 (P2); no longer R12.2
- net at Q1.3 (C), Q2.3 (C), Q3.3 (C): now also JP1.1; no longer C8.2, Q10.2 (B)
- net at Q12.1 (E): now also RV1.1
- new net: C3.2, R10.2, R5.2, R8.2
- new net: C8.2, JP1.2, Q10.2 (B)
- new net: R15.1, RV1.2, RV1.3
- new net FBACK: R12.2
Other:
- note added: "Conectores\n"
- note added: "Power Flags\n"

Commit message: Termino la primera version del PCB para el amplificador, queda engordar las pistas que llevan alta corriente.
Parts:
- CON1: footprint (none) -> Connect:BARREL_JACK
- JP1, P1, P2, P3, P4: footprint Socket_Strips:Socket_Strip_Angled_1x02 -> Socket_Strips:Socket_Strip_Straight_1x02
- P5: footprint (none) -> Pin_Headers:Pin_Header_Straight_1x02
- R1, R10, R11, R12, R13, R14, R15, R2, R3, R4, R5, R6, R7, R8, R9: footprint Resistors_SMD:R_0603_HandSoldering -> Resistors_ThroughHole:Resistor_Horizontal_RM10mm
- RV1: footprint (none) -> Pin_Headers:Pin_Header_Straight_1x03
Connections:
- net +VA: now also C6.2
- net -VA: now also C5.1, R10.1, R14.2, R15.2
- net GND: now also C5.2, C6.1; no longer R10.1, R14.2, R15.2
- net at C3.2, R10.2, R5.2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: now also C4.1
Other:
- moved on the sheet: C6

Commit message: Arreglo problema, se mostraba cobre en el front , solo lo hice para Q1, queda hacerlo en todos y ajustar bien los drills, acorde a los que existen en el LCI...
Parts:
- Q1: footprint Transistors_TO-220:TO-220_Neutral123_Vertical -> pcb:TRANSISTOR_PARA_GCLASS
Changed lines of the file:
@@
 EESchema Schematic File Version 2
+LIBS:lib_ampli
 LIBS:power
 LIBS:device
@@
 F 0 "Q1" H 3250 4200 50  0000 R CNN
 F 1 "MPSA56_PNP_EBC" H 3300 3900 50  0000 R CNN
-F 2 "Transistors_TO-220:TO-220_Neutral123_Vertical" H 3150 4250 29  0001 C CNN
+F 2 "pcb:TRANSISTOR_PARA_GCLASS" H 3150 4250 29  0001 C CNN
 F 3 "" H 2950 4150 60  0000 C CNN
 	1    2950 4150

Commit message: Cambio footprints, empiezo a re-rutear
Parts:
- removed JP1: JUMPER, Socket_Strips:Socket_Strip_Straight_1x02, symbol JUMPER
- added P6: CONN_01X01, Pin_Headers:Pin_Header_Straight_1x03, symbol CONN_01X01
- Q1: footprint pcb:TRANSISTOR_PARA_GCLASS -> pcb:MPSA06-56_TO92_EBC
- Q10, Q11, Q12, Q2, Q3, Q4, Q5, Q6, Q7, Q8, Q9: footprint Transistors_TO-220:TO-220_Neutral123_Vertical -> pcb:MPSA06-56_TO92_EBC
Connections:
- net at Q1.3 (C), Q2.3 (C), Q3.3 (C): now also C8.2, Q10.2 (B), P6.1 (P1)
Changed lines of the file:
@@
 F 0 "Q6" H 5400 1950 50  0000 R CNN
 F 1 "MPSA56_PNP_EBC" H 5550 1650 50  0000 R CNN
-F 2 "Transistors_TO-220:TO-220_Neutral123_Vertical" H 5300 2000 29  0001 C CNN
+F 2 "pcb:MPSA06-56_TO92_EBC" H 5300 2000 29  0001 C CNN
 F 3 "" H 5100 1900 60  0000 C CNN
 	1    5100 1900
@@
 F 0 "Q3" H 4150 5000 50  0000 R CNN
 F 1 "MPSA06_NPN_EBC" H 4250 4700 50  0000 R CNN
-F 2 "Transistors_TO-220:TO-220_Neutral123_Vertical" H 4050 5050 29  0001 C CNN
+F 2 "pcb:MPSA06-56_TO92_EBC" H 4050 5050 29  0001 C CNN
 F 3 "" H 3850 4950 60  0000 C CNN
 	1    3850 4950
@@
 F 0 "Q5" H 5300 5000 50  0000 R CNN
 F 1 "MPSA06_NPN_EBC" H 5500 4700 50  0000 R CNN
-F 2 "Transistors_TO-220:TO-220_Neutral123_Vertical" H 5200 5050 29  0001 C CNN
+F 2 "pcb:MPSA06-56_TO92_EBC" H 5200 5050 29  0001 C CNN
 F 3 "" H 5000 4950 60  0000 C CNN
 	1    5000 4950
@@
 F 0 "Q9" H 7950 1950 50  0000 R CNN
 F 1 "MPSA56_PNP_EBC" H 8050 1700 50  0000 R CNN
-F 2 "Transistors_TO-220:TO-220_Neutral123_Vertical" H 7850 2000 29  0001 C CNN
+F 2 "pcb:MPSA06-56_TO92_EBC" H 7850 2000 29  0001 C CNN
 F 3 "" H 7650 1900 60  0000 C CNN
 	1    7650 1900
@@
 F 0 "Q4" H 4750 1950 50  0000 R CNN
 F 1 "MPSA56_PNP_EBC" H 4850 1650 50  0000 R CNN
-F 2 "Transistors_TO-220:TO-220_Neutral123_Vertical" H 4650 2000 29  0001 C CNN
+F 2 "pcb:MPSA06-56_TO92_EBC" H 4650 2000 29  0001 C CNN
 F 3 "" H 4450 1900 60  0000 C CNN
 	1    4450 1900
@@
 F 0 "Q7" H 5500 4200 50  0000 R CNN
 F 1 "MPSA56_PNP_EBC" H 5750 3900 50  0000 R CNN
-F 2 "Transistors_TO-220:TO-220_Neutral123_Vertical" H 5400 4250 29  0001 C CNN
+F 2 "pcb:MPSA06-56_TO92_EBC" H 5400 4250 29  0001 C CNN
 F 3 "" H 5200 4150 60  0000 C CNN
 	1    5200 4150
@@
 F 0 "Q8" H 6200 4200 50  0000 R CNN
 F 1 "MPSA56_PNP_EBC" H 6250 3900 50  0000 R CNN
-F 2 "Transistors_TO-220:TO-220_Neutral123_Vertical" H 6100 4250 29  0001 C CNN
+F 2 "pcb:MPSA06-56_TO92_EBC" H 6100 4250 29  0001 C CNN
 F 3 "" H 5900 4150 60  0000 C CNN
 	1    5900 4150
@@
 F 0 "Q2" H 3950 4200 50  0000 R CNN
 F 1 "MPSA56_PNP_EBC" H 4050 3900 50  0000 R CNN
-F 2 "Transistors_TO-220:TO-220_Neutral123_Vertical" H 3850 4250 29  0001 C CNN
+F 2 "pcb:MPSA06-56_TO92_EBC" H 3850 4250 29  0001 C CNN
 F 3 "" H 3650 4150 60  0000 C CNN
 	1    3650 4150
@@
 F 0 "Q1" H 3250 4200 50  0000 R CNN
 F 1 "MPSA56_PNP_EBC" H 3300 3900 50  0000 R CNN
-F 2 "pcb:TRANSISTOR_PARA_GCLASS" H 3150 4250 29  0001 C CNN
+F 2 "pcb:MPSA06-56_TO92_EBC" H 3150 4250 29  0001 C CNN
 F 3 "" H 2950 4150 60  0000 C CNN
 	1    2950 4150
@@
 F 0 "Q11" H 8600 1950 50  0000 R CNN
 F 1 "MPSA56_PNP_EBC" H 8750 1700 50  0000 R CNN
-F 2 "Transistors_TO-220:TO-220_Neutral123_Vertical" H 8500 2000 29  0001 C CNN
+F 2 "pcb:MPSA06-56_TO92_EBC" H 8500 2000 29  0001 C CNN
 F 3 "" H 8300 1900 60  0000 C CNN
 	1    8300 1900
@@
 F 0 "Q10" H 8000 4550 50  0000 R CNN
 F 1 "MPSA06_NPN_EBC" H 8250 4250 50  0000 R CNN
-F 2 "Transistors_TO-220:TO-220_Neutral123_Vertical" H 7900 4600 29  0001 C CNN
+F 2 "pcb:MPSA06-56_TO92_EBC" H 7900 4600 29  0001 C CNN
 F 3 "" H 7700 4500 60  0000 C CNN
 	1    7700 4500
@@
 F 0 "Q12" H 8600 4200 50  0000 R CNN
 F 1 "MPSA06_NPN_EBC" H 8800 3950 50  0000 R CNN
-F 2 "Transistors_TO-220:TO-220_Neutral123_Vertical" H 8500 4250 29  0001 C CNN
+F 2 "pcb:MPSA06-56_TO92_EBC" H 8500 4250 29  0001 C CNN
 F 3 "" H 8300 4150 60  0000 C CNN
 	1    8300 4150
@@
 	1    0    0    -1
 $EndComp
-$Comp
-L JUMPER JP1
-U 1 1 556CD613
-P 6950 4250
-F 0 "JP1" H 6950 4400 50  0000 C CNN
-F 1 "JUMPER" H 6950 4170 50  0000 C CNN
-F 2 "Socket_Strips:Socket_Strip_Straight_1x02" H 6950 4250 60  0001 C CNN
-F 3 "" H 6950 4250 60  0000 C CNN
-	1    6950 4250
-	1    0    0    -1
-$EndComp
-Wire Wire Line
-	7250 4500 7500 4500
-Wire Wire Line
-	7250 4250 7250 4500
-Wire Wire Line
-	6650 4250 6650 4500
-Wire Wire Line
-	6650 4500 3750 4500
+Wire Wire Line
+	3750 4500 7500 4500
 $Comp
 L POT RV1
@@
 Wire Wire Line
 	6100 2050 6100 1950
+Wire Wire Line
+	7050 4500 7050 4300
+Connection ~ 7050 4500
+$Comp
+L CONN_01X01 P6
+U 1 1 55768354
+P 6850 4300
+F 0 "P6" H 6850 4400 50  0000 C CNN
+F 1 "CONN_01X01" H 6850 4150 50  0000 C CNN
+F 2 "Pin_Headers:Pin_Header_Straight_1x03" H 6850 4300 60  0001 C CNN
+F 3 "" H 6850 4300 60  0000 C CNN
+	1    6850 4300
+	-1   0    0    1
+$EndComp
 $EndSCHEMATC

Commit message: nacho la soba
Parts:
- P6: footprint Pin_Headers:Pin_Header_Straight_1x03 -> Pin_Headers:Pin_Header_Straight_1x01
Connections:
- net GND: now also C3.1
Changed lines of the file:
@@
 L GND #PWR028
 U 1 1 556CC461
-P 5100 6150
-F 0 "#PWR028" H 5100 5900 50  0001 C CNN
-F 1 "GND" H 5100 6000 50  0000 C CNN
-F 2 "" H 5100 6150 60  0000 C CNN
-F 3 "" H 5100 6150 60  0000 C CNN
-	1    5100 6150
+P 5100 6300
+F 0 "#PWR028" H 5100 6050 50  0001 C CNN
+F 1 "GND" H 5100 6150 50  0000 C CNN
+F 2 "" H 5100 6300 60  0000 C CNN
+F 3 "" H 5100 6300 60  0000 C CNN
+	1    5100 6300
 	1    0    0    -1
 $EndComp
@@
 F 0 "P6" H 6850 4400 50  0000 C CNN
 F 1 "CONN_01X01" H 6850 4150 50  0000 C CNN
-F 2 "Pin_Headers:Pin_Header_Straight_1x03" H 6850 4300 60  0001 C CNN
+F 2 "Pin_Headers:Pin_Header_Straight_1x01" H 6850 4300 60  0001 C CNN
 F 3 "" H 6850 4300 60  0000 C CNN
 	1    6850 4300
 	-1   0    0    1
 $EndComp
+Wire Wire Line
+	5100 6200 5100 6300
 $EndSCHEMATC
