File: pcb/amplificador_gclass.sch (KiCad schematic (older format))
At the start: 43 parts, among them CON1 AUDIO_IN, P1 +VA_GND, P2 +VB_GND, P3 -VA_GND, P4 -VB_GND, P5 OUT, P6 CONN_01X01, Q1 MPSA56_PNP_EBC, Q10 MPSA06_NPN_EBC, Q11 MPSA56_PNP_EBC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

Commit message: ultimos avances falta poco para terminar
Changed lines of the file:
@@
 L GND #PWR014
 U 1 1 555F1530
-P 6500 5450
-F 0 "#PWR014" H 6500 5200 50  0001 C CNN
-F 1 "GND" H 6500 5300 50  0000 C CNN
-F 2 "" H 6500 5450 60  0000 C CNN
-F 3 "" H 6500 5450 60  0000 C CNN
-	1    6500 5450
+P 6500 5550
+F 0 "#PWR014" H 6500 5300 50  0001 C CNN
+F 1 "GND" H 6500 5400 50  0000 C CNN
+F 2 "" H 6500 5550 60  0000 C CNN
+F 3 "" H 6500 5550 60  0000 C CNN
+	1    6500 5550
 	1    0    0    -1
 $EndComp
@@
 Wire Wire Line
 	5100 6200 5100 6300
+Wire Wire Line
+	6500 5450 6500 5550
 $EndSCHEMATC

Commit message: pcb casi listo
el pcb esta casi listo
Parts:
- added P13, P14, P15, P16, P17, P18: CONN_01X01, Pin_Headers:Pin_Header_Straight_1x01, symbol CONN_01X01
Connections:
- net GND: now also P13.1 (P1), P14.1 (P1), P15.1 (P1), P16.1 (P1), P17.1 (P1), P18.1 (P1)
Changed lines of the file:
@@
 Wire Wire Line
 	6500 5450 6500 5550
+$Comp
+L CONN_01X01 P13
+U 1 1 55779C41
+P 1250 6100
+F 0 "P13" H 1250 6200 50  0000 C CNN
+F 1 "CONN_01X01" H 1250 5950 50  0000 C CNN
+F 2 "Pin_Headers:Pin_Header_Straight_1x01" H 1250 6100 60  0001 C CNN
+F 3 "" H 1250 6100 60  0000 C CNN
+	1    1250 6100
+	-1   0    0    1
+$EndComp
+$Comp
+L CONN_01X01 P14
+U 1 1 5577A4C3
+P 1250 6500
+F 0 "P14" H 1250 6600 50  0000 C CNN
+F 1 "CONN_01X01" H 1250 6350 50  0000 C CNN
+F 2 "Pin_Headers:Pin_Header_Straight_1x01" H 1250 6500 60  0001 C CNN
+F 3 "" H 1250 6500 60  0000 C CNN
+	1    1250 6500
+	-1   0    0    1
+$EndComp
+$Comp
+L GND #PWR031
+U 1 1 5577AAD9
+P 1550 6150
+F 0 "#PWR031" H 1550 5900 50  0001 C CNN
+F 1 "GND" H 1550 6000 50  0000 C CNN
+F 2 "" H 1550 6150 60  0000 C CNN
+F 3 "" H 1550 6150 60  0000 C CNN
+	1    1550 6150
+	1    0    0    -1
+$EndComp
+$Comp
+L GND #PWR032
+U 1 1 5577B1BF
+P 1550 6550
+F 0 "#PWR032" H 1550 6300 50  0001 C CNN
+F 1 "GND" H 1550 6400 50  0000 C CNN
+F 2 "" H 1550 6550 60  0000 C CNN
+F 3 "" H 1550 6550 60  0000 C CNN
+	1    1550 6550
+	1    0    0    -1
+$EndComp
+Wire Wire Line
+	1450 6500 1550 6500
+Wire Wire Line
+	1550 6500 1550 6550
+Wire Wire Line
+	1550 6150 1550 6100
+Wire Wire Line
+	1550 6100 1450 6100
+$Comp
+L CONN_01X01 P15
+U 1 1 5577CF3C
+P 1250 6950
+F 0 "P15" H 1250 7050 50  0000 C CNN
+F 1 "CONN_01X01" H 1250 6800 50  0000 C CNN
+F 2 "Pin_Headers:Pin_Header_Straight_1x01" H 1250 6950 60  0001 C CNN
+F 3 "" H 1250 6950 60  0000 C CNN
+	1    1250 6950
+	-1   0    0    1
+$EndComp
+$Comp
+L GND #PWR033
+U 1 1 5577D0A0
+P 1550 7000
+F 0 "#PWR033" H 1550 6750 50  0001 C CNN
+F 1 "GND" H 1550 6850 50  0000 C CNN
+F 2 "" H 1550 7000 60  0000 C CNN
+F 3 "" H 1550 7000 60  0000 C CNN
+	1    1550 7000
+	1    0    0    -1
+$EndComp
+Wire Wire Line
+	1450 6950 1550 6950
+Wire Wire Line
+	1550 6950 1550 7000
+$Comp
+L CONN_01X01 P16
+U 1 1 5577D35E
+P 1250 7400
+F 0 "P16" H 1250 7500 50  0000 C CNN
+F 1 "CONN_01X01" H 1250 7250 50  0000 C CNN
+F 2 "Pin_Headers:Pin_Header_Straight_1x01" H 1250 7400 60  0001 C CNN
+F 3 "" H 1250 7400 60  0000 C CNN
+	1    1250 7400
+	-1   0    0    1
+$EndComp
+$Comp
+L CONN_01X01 P17
+U 1 1 5577D3D8
+P 2100 7400
+F 0 "P17" H 2100 7500 50  0000 C CNN
+F 1 "CONN_01X01" H 2100 7250 50  0000 C CNN
+F 2 "Pin_Headers:Pin_Header_Straight_1x01" H 2100 7400 60  0001 C CNN
+F 3 "" H 2100 7400 60  0000 C CNN
+	1    2100 7400
+	-1   0    0    1
+$EndComp
+$Comp
+L GND #PWR034
+U 1 1 5577D464
+P 1550 7450
+F 0 "#PWR034" H 1550 7200 50  0001 C CNN
+F 1 "GND" H 1550 7300 50  0000 C CNN
+F 2 "" H 1550 7450 60  0000 C CNN
+F 3 "" H 1550 7450 60  0000 C CNN
+	1    1550 7450
+	1    0    0    -1
+$EndComp
+$Comp
+L GND #PWR035
+U 1 1 5577D4CF
+P 2400 7450
+F 0 "#PWR035" H 2400 7200 50  0001 C CNN
+F 1 "GND" H 2400 7300 50  0000 C CNN
+F 2 "" H 2400 7450 60  0000 C CNN
+F 3 "" H 2400 7450 60  0000 C CNN
+	1    2400 7450
+	1    0    0    -1
+$EndComp
+Wire Wire Line
+	2400 7450 2400 7400
+Wire Wire Line
+	2400 7400 2300 7400
+Wire Wire Line
+	1550 7450 1550 7400
+Wire Wire Line
+	1550 7400 1450 7400
+$Comp
+L CONN_01X01 P18
+U 1 1 5577E7A1
+P 2100 6800
+F 0 "P18" H 2100 6900 50  0000 C CNN
+F 1 "CONN_01X01" H 2100 6650 50  0000 C CNN
+F 2 "Pin_Headers:Pin_Header_Straight_1x01" H 2100 6800 60  0001 C CNN
+F 3 "" H 2100 6800 60  0000 C CNN
+	1    2100 6800
+	-1   0    0    1
+$EndComp
+$Comp
+L GND #PWR036
+U 1 1 5577E81F
+P 2400 6850
+F 0 "#PWR036" H 2400 6600 50  0001 C CNN
+F 1 "GND" H 2400 6700 50  0000 C CNN
+F 2 "" H 2400 6850 60  0000 C CNN
+F 3 "" H 2400 6850 60  0000 C CNN
+	1    2400 6850
+	1    0    0    -1
+$EndComp
+Wire Wire Line
+	2400 6850 2400 6800
+Wire Wire Line
+	2400 6800 2300 6800
 $EndSCHEMATC

Commit message: cambios
Parts:
- added P9: CONN_01X01, pcb:bornera_grande, symbol CONN_01X01
- P1: renamed from P13; footprint Pin_Headers:Pin_Header_Straight_1x01 -> Socket_Strips:Socket_Strip_Straight_1x02
- P10: renamed from P18; footprint Pin_Headers:Pin_Header_Straight_1x01 -> pcb:bornera_grande
- P11: renamed from P17; footprint Pin_Headers:Pin_Header_Straight_1x01 -> pcb:bornera_grande
- P12: renamed from P5; footprint Pin_Headers:Pin_Header_Straight_1x02 -> pcb:bornera_grande
- P2: renamed from P14; footprint Pin_Headers:Pin_Header_Straight_1x01 -> Socket_Strips:Socket_Strip_Straight_1x02
- P3: renamed from P15; footprint Pin_Headers:Pin_Header_Straight_1x01 -> Socket_Strips:Socket_Strip_Straight_1x02
- P4: renamed from P16; footprint Pin_Headers:Pin_Header_Straight_1x01 -> Socket_Strips:Socket_Strip_Straight_1x02
- P5: renamed from P1; footprint Socket_Strips:Socket_Strip_Straight_1x02 -> Pin_Headers:Pin_Header_Straight_1x02
- P6: renamed from P2; footprint Socket_Strips:Socket_Strip_Straight_1x02 -> Pin_Headers:Pin_Header_Straight_1x01
- P7: renamed from P3; footprint Socket_Strips:Socket_Strip_Straight_1x02 -> pcb:bornera_chica
- P8: renamed from P4; footprint Socket_Strips:Socket_Strip_Straight_1x02 -> pcb:bornera_chica
- renumbered P6 to P13
Connections:
- net GND: now also P9.1 (P1)
Changed lines of the file:
@@
 $Descr A4 11693 8268
 encoding utf-8
-Sheet 1 2
+Sheet 1 3
 Title "Amplificador Clase G "
 Date "Mon 01 Jun 2015"
@@
 $EndComp
 $Comp
-L CONN_01X02 P4
+L CONN_01X02 P8
 U 1 1 555EA185
 P 2000 3250
-F 0 "P4" H 2000 3400 50  0000 C CNN
+F 0 "P8" H 2000 3400 50  0000 C CNN
 F 1 "-VB_GND" V 2100 3250 50  0000 C CNN
-F 2 "Socket_Strips:Socket_Strip_Straight_1x02" H 2000 3250 60  0001 C CNN
+F 2 "pcb:bornera_chica" H 2000 3250 60  0001 C CNN
 F 3 "" H 2000 3250 60  0000 C CNN
 	1    2000 3250
@@
 $EndComp
 $Comp
-L CONN_01X02 P2
+L CONN_01X02 P6
 U 1 1 555EA18B
 P 1450 3250
-F 0 "P2" H 1450 3400 50  0000 C CNN
+F 0 "P6" H 1450 3400 50  0000 C CNN
 F 1 "+VB_GND" V 1550 3250 50  0000 C CNN
-F 2 "Socket_Strips:Socket_Strip_Straight_1x02" H 1450 3250 60  0001 C CNN
+F 2 "Pin_Headers:Pin_Header_Straight_1x01" H 1450 3250 60  0001 C CNN
 F 3 "" H 1450 3250 60  0000 C CNN
 	1    1450 3250
@@
 $EndComp
 $Comp
-L CONN_01X02 P1
+L CONN_01X02 P5
 U 1 1 555E9A30
 P 1450 2350
-F 0 "P1" H 1450 2500 50  0000 C CNN
+F 0 "P5" H 1450 2500 50  0000 C CNN
 F 1 "+VA_GND" V 1550 2350 50  0000 C CNN
-F 2 "Socket_Strips:Socket_Strip_Straight_1x02" H 1450 2350 60  0001 C CNN
+F 2 "Pin_Headers:Pin_Header_Straight_1x02" H 1450 2350 60  0001 C CNN
 F 3 "" H 1450 2350 60  0000 C CNN
 	1    1450 2350
@@
 $EndComp
 $Comp
-L CONN_01X02 P3
+L CONN_01X02 P7
 U 1 1 555E9943
 P 2000 2350
-F 0 "P3" H 2000 2500 50  0000 C CNN
+F 0 "P7" H 2000 2500 50  0000 C CNN
 F 1 "-VA_GND" V 2100 2350 50  0000 C CNN
-F 2 "Socket_Strips:Socket_Strip_Straight_1x02" H 2000 2350 60  0001 C CNN
+F 2 "pcb:bornera_chica" H 2000 2350 60  0001 C CNN
 F 3 "" H 2000 2350 60  0000 C CNN
 	1    2000 2350
@@
 	8550 5300 8550 5050
 $Comp
-L CONN_01X02 P5
+L CONN_01X02 P12
 U 1 1 556D3736
 P 2600 3200
-F 0 "P5" H 2600 3350 50  0000 C CNN
+F 0 "P12" H 2600 3350 50  0000 C CNN
 F 1 "OUT" V 2700 3200 50  0000 C CNN
-F 2 "Pin_Headers:Pin_Header_Straight_1x02" H 2600 3200 60  0001 C CNN
+F 2 "pcb:bornera_grande" H 2600 3200 60  0001 C CNN
 F 3 "" H 2600 3200 60  0000 C CNN
 	1    2600 3200
@@
 Connection ~ 7050 4500
 $Comp
-L CONN_01X01 P6
+L CONN_01X01 P13
 U 1 1 55768354
 P 6850 4300
-F 0 "P6" H 6850 4400 50  0000 C CNN
+F 0 "P13" H 6850 4400 50  0000 C CNN
 F 1 "CONN_01X01" H 6850 4150 50  0000 C CNN
 F 2 "Pin_Headers:Pin_Header_Straight_1x01" H 6850 4300 60  0001 C CNN
@@
 	6500 5450 6500 5550
 $Comp
-L CONN_01X01 P13
+L CONN_01X01 P1
 U 1 1 55779C41
 P 1250 6100
-F 0 "P13" H 1250 6200 50  0000 C CNN
+F 0 "P1" H 1250 6200 50  0000 C CNN
 F 1 "CONN_01X01" H 1250 5950 50  0000 C CNN
-F 2 "Pin_Headers:Pin_Header_Straight_1x01" H 1250 6100 60  0001 C CNN
+F 2 "Socket_Strips:Socket_Strip_Straight_1x02" H 1250 6100 60  0001 C CNN
 F 3 "" H 1250 6100 60  0000 C CNN
 	1    1250 6100
@@
 $EndComp
 $Comp
-L CONN_01X01 P14
+L CONN_01X01 P2
 U 1 1 5577A4C3
 P 1250 6500
-F 0 "P14" H 1250 6600 50  0000 C CNN
+F 0 "P2" H 1250 6600 50  0000 C CNN
 F 1 "CONN_01X01" H 1250 6350 50  0000 C CNN
-F 2 "Pin_Headers:Pin_Header_Straight_1x01" H 1250 6500 60  0001 C CNN
+F 2 "Socket_Strips:Socket_Strip_Straight_1x02" H 1250 6500 60  0001 C CNN
 F 3 "" H 1250 6500 60  0000 C CNN
 	1    1250 6500
@@
 	1550 6100 1450 6100
 $Comp
-L CONN_01X01 P15
+L CONN_01X01 P3
 U 1 1 5577CF3C
 P 1250 6950
-F 0 "P15" H 1250 7050 50  0000 C CNN
+F 0 "P3" H 1250 7050 50  0000 C CNN
 F 1 "CONN_01X01" H 1250 6800 50  0000 C CNN
-F 2 "Pin_Headers:Pin_Header_Straight_1x01" H 1250 6950 60  0001 C CNN
+F 2 "Socket_Strips:Socket_Strip_Straight_1x02" H 1250 6950 60  0001 C CNN
 F 3 "" H 1250 6950 60  0000 C CNN
 	1    1250 6950
@@
 	1550 6950 1550 7000
 $Comp
-L CONN_01X01 P16
+L CONN_01X01 P4
 U 1 1 5577D35E
 P 1250 7400
-F 0 "P16" H 1250 7500 50  0000 C CNN
+F 0 "P4" H 1250 7500 50  0000 C CNN
 F 1 "CONN_01X01" H 1250 7250 50  0000 C CNN
-F 2 "Pin_Headers:Pin_Header_Straight_1x01" H 1250 7400 60  0001 C CNN
+F 2 "Socket_Strips:Socket_Strip_Straight_1x02" H 1250 7400 60  0001 C CNN
 F 3 "" H 1250 7400 60  0000 C CNN
 	1    1250 7400
@@
 $EndComp
 $Comp
-L CONN_01X01 P17
+L CONN_01X01 P11
 U 1 1 5577D3D8
 P 2100 7400
-F 0 "P17" H 2100 7500 50  0000 C CNN
+F 0 "P11" H 2100 7500 50  0000 C CNN
 F 1 "CONN_01X01" H 2100 7250 50  0000 C CNN
-F 2 "Pin_Headers:Pin_Header_Straight_1x01" H 2100 7400 60  0001 C CNN
+F 2 "pcb:bornera_grande" H 2100 7400 60  0001 C CNN
 F 3 "" H 2100 7400 60  0000 C CNN
 	1    2100 7400
@@
 	1550 7400 1450 7400
 $Comp
-L CONN_01X01 P18
+L CONN_01X01 P10
 U 1 1 5577E7A1
 P 2100 6800
-F 0 "P18" H 2100 6900 50  0000 C CNN
+F 0 "P10" H 2100 6900 50  0000 C CNN
 F 1 "CONN_01X01" H 2100 6650 50  0000 C CNN
-F 2 "Pin_Headers:Pin_Header_Straight_1x01" H 2100 6800 60  0001 C CNN
+F 2 "pcb:bornera_grande" H 2100 6800 60  0001 C CNN
 F 3 "" H 2100 6800 60  0000 C CNN
 	1    2100 6800
@@
 Wire Wire Line
 	2400 6800 2300 6800
+$Comp
+L CONN_01X01 P9
+U 1 1 5579C4A9
+P 2100 6100
+F 0 "P9" H 2100 6200 50  0000 C CNN
+F 1 "CONN_01X01" H 2100 5950 50  0000 C CNN
+F 2 "pcb:bornera_grande" H 2100 6100 60  0001 C CNN
+F 3 "" H 2100 6100 60  0000 C CNN
+	1    2100 6100
+	-1   0    0    1
+$EndComp
+$Comp
+L GND #PWR037
+U 1 1 5579C52B
+P 2400 6150
+F 0 "#PWR037" H 2400 5900 50  0001 C CNN
+F 1 "GND" H 2400 6000 50  0000 C CNN
+F 2 "" H 2400 6150 60  0000 C CNN
+F 3 "" H 2400 6150 60  0000 C CNN
+	1    2400 6150
+	1    0    0    -1
+$EndComp
+Wire Wire Line
+	2300 6100 2400 6100
+Wire Wire Line
+	2400 6100 2400 6150
 $EndSCHEMATC

Commit message: pcb terminado
Parts:
- removed CON1: AUDIO_IN, Connect:BARREL_JACK, symbol BARREL_JACK
- removed P11: CONN_01X01, pcb:bornera_grande, symbol CONN_01X01
- added J?: Jack_3.5mm_5pin, symbol Jack_3.5mm_5pin
Connections:
- net GND: now also J?.1 (S), J?.3 (R), J?.5 (RS)
- net IN: now also J?.2 (T), J?.4 (TS)
Changed lines of the file:
@@
 LIBS:contrib
 LIBS:valves
+LIBS:w_connectors
 LIBS:amplificador_gclass-cache
 EELAYER 25 0
@@
 	0    -1   -1   0
 $EndComp
-$Comp
-L BARREL_JACK CON1
-U 1 1 556D4923
-P 2900 2450
-F 0 "CON1" H 2900 2700 60  0000 C CNN
-F 1 "AUDIO_IN" H 2900 2250 60  0000 C CNN
-F 2 "Connect:BARREL_JACK" H 2900 2450 60  0001 C CNN
-F 3 "" H 2900 2450 60  0000 C CNN
-	1    2900 2450
-	-1   0    0    1
-$EndComp
 Wire Wire Line
 	2400 2250 2500 2250
@@
 	2500 2250 2500 2350
 Wire Wire Line
-	2500 2350 2600 2350
+	2500 2350 2850 2350
 Wire Wire Line
 	2600 2350 2600 2450
@@
 $EndComp
 $Comp
-L CONN_01X01 P11
-U 1 1 5577D3D8
-P 2100 7400
-F 0 "P11" H 2100 7500 50  0000 C CNN
-F 1 "CONN_01X01" H 2100 7250 50  0000 C CNN
-F 2 "pcb:bornera_grande" H 2100 7400 60  0001 C CNN
-F 3 "" H 2100 7400 60  0000 C CNN
-	1    2100 7400
-	-1   0    0    1
-$EndComp
-$Comp
 L GND #PWR034
 U 1 1 5577D464
@@
 	1    0    0    -1
 $EndComp
-$Comp
-L GND #PWR035
-U 1 1 5577D4CF
-P 2400 7450
-F 0 "#PWR035" H 2400 7200 50  0001 C CNN
-F 1 "GND" H 2400 7300 50  0000 C CNN
-F 2 "" H 2400 7450 60  0000 C CNN
-F 3 "" H 2400 7450 60  0000 C CNN
-	1    2400 7450
-	1    0    0    -1
-$EndComp
-Wire Wire Line
-	2400 7450 2400 7400
-Wire Wire Line
-	2400 7400 2300 7400
 Wire Wire Line
 	1550 7450 1550 7400
@@
 $EndComp
 $Comp
-L GND #PWR036
+L GND #PWR035
 U 1 1 5577E81F
 P 2400 6850
-F 0 "#PWR036" H 2400 6600 50  0001 C CNN
+F 0 "#PWR035" H 2400 6600 50  0001 C CNN
 F 1 "GND" H 2400 6700 50  0000 C CNN
 F 2 "" H 2400 6850 60  0000 C CNN
@@
 $EndComp
 $Comp
-L GND #PWR037
+L GND #PWR036
 U 1 1 5579C52B
 P 2400 6150
-F 0 "#PWR037" H 2400 5900 50  0001 C CNN
+F 0 "#PWR036" H 2400 5900 50  0001 C CNN
 F 1 "GND" H 2400 6000 50  0000 C CNN
 F 2 "" H 2400 6150 60  0000 C CNN
@@
 Wire Wire Line
 	2400 6100 2400 6150
+$Comp
+L Jack_3.5mm_5pin J?
+U 1 1 557AAF8F
+P 3000 2550
+F 0 "J?" H 3000 2800 60  0000 C CNN
+F 1 "Jack_3.5mm_5pin" H 3000 2250 60  0000 C CNN
+F 2 "" H 3000 2600 60  0000 C CNN
+F 3 "" H 3000 2600 60  0000 C CNN
+	1    3000 2550
+	1    0    0    -1
+$EndComp
+Connection ~ 2600 2350
+Wire Wire Line
+	2600 2450 2400 2450
+Wire Wire Line
+	2400 2450 2400 2750
+Wire Wire Line
+	2400 2750 2850 2750
+Wire Wire Line
+	2750 2750 2750 2650
+Wire Wire Line
+	2750 2650 2850 2650
+Connection ~ 2750 2750
+Wire Wire Line
+	2850 2550 2600 2550
+Wire Wire Line
+	2850 2450 2800 2450
+Wire Wire Line
+	2800 2450 2800 2550
+Connection ~ 2800 2550
 $EndSCHEMATC

Commit message: ahora si terminado
Parts:
- J1: renamed from J?; footprint (none) -> pcb:jack_puto
- P1, P2, P3, P4: footprint Socket_Strips:Socket_Strip_Straight_1x02 -> Pin_Headers:Pin_Header_Straight_1x01
- P10, P9: footprint pcb:bornera_grande -> Pin_Headers:Pin_Header_Straight_1x01
- P12: footprint pcb:bornera_grande -> Pin_Headers:Pin_Header_Straight_1x02
- P6: footprint Pin_Headers:Pin_Header_Straight_1x01 -> Pin_Headers:Pin_Header_Straight_1x02
- P7, P8: footprint pcb:bornera_chica -> Pin_Headers:Pin_Header_Straight_1x02
Connections:
- net GND: now also J1.4 (TS); no longer J1.3 (R)
- net IN: now also J1.3 (R); no longer J1.2 (T), J1.4 (TS)
- no-connect marks 0 -> 1
Changed lines of the file:
@@
 F 0 "P8" H 2000 3400 50  0000 C CNN
 F 1 "-VB_GND" V 2100 3250 50  0000 C CNN
-F 2 "pcb:bornera_chica" H 2000 3250 60  0001 C CNN
+F 2 "Pin_Headers:Pin_Header_Straight_1x02" H 2000 3250 60  0001 C CNN
 F 3 "" H 2000 3250 60  0000 C CNN
 	1    2000 3250
@@
 F 0 "P6" H 1450 3400 50  0000 C CNN
 F 1 "+VB_GND" V 1550 3250 50  0000 C CNN
-F 2 "Pin_Headers:Pin_Header_Straight_1x01" H 1450 3250 60  0001 C CNN
+F 2 "Pin_Headers:Pin_Header_Straight_1x02" H 1450 3250 60  0001 C CNN
 F 3 "" H 1450 3250 60  0000 C CNN
 	1    1450 3250
@@
 F 0 "P7" H 2000 2500 50  0000 C CNN
 F 1 "-VA_GND" V 2100 2350 50  0000 C CNN
-F 2 "pcb:bornera_chica" H 2000 2350 60  0001 C CNN
+F 2 "Pin_Headers:Pin_Header_Straight_1x02" H 2000 2350 60  0001 C CNN
 F 3 "" H 2000 2350 60  0000 C CNN
 	1    2000 2350
@@
 Wire Notes Line
 	2800 1800 2800 1000
-Text GLabel 2600 2550 0    60   Input ~ 0
+Text GLabel 2750 2650 0    60   Input ~ 0
 IN
 $Comp
@@
 F 0 "P12" H 2600 3350 50  0000 C CNN
 F 1 "OUT" V 2700 3200 50  0000 C CNN
-F 2 "pcb:bornera_grande" H 2600 3200 60  0001 C CNN
+F 2 "Pin_Headers:Pin_Header_Straight_1x02" H 2600 3200 60  0001 C CNN
 F 3 "" H 2600 3200 60  0000 C CNN
 	1    2600 3200
@@
 Wire Wire Line
 	2500 2350 2850 2350
-Wire Wire Line
-	2600 2350 2600 2450
 Wire Notes Line
 	3400 3700 3400 2100
@@
 F 0 "P1" H 1250 6200 50  0000 C CNN
 F 1 "CONN_01X01" H 1250 5950 50  0000 C CNN
-F 2 "Socket_Strips:Socket_Strip_Straight_1x02" H 1250 6100 60  0001 C CNN
+F 2 "Pin_Headers:Pin_Header_Straight_1x01" H 1250 6100 60  0001 C CNN
 F 3 "" H 1250 6100 60  0000 C CNN
 	1    1250 6100
@@
 F 0 "P2" H 1250 6600 50  0000 C CNN
 F 1 "CONN_01X01" H 1250 6350 50  0000 C CNN
-F 2 "Socket_Strips:Socket_Strip_Straight_1x02" H 1250 6500 60  0001 C CNN
+F 2 "Pin_Headers:Pin_Header_Straight_1x01" H 1250 6500 60  0001 C CNN
 F 3 "" H 1250 6500 60  0000 C CNN
 	1    1250 6500
@@
 F 0 "P3" H 1250 7050 50  0000 C CNN
 F 1 "CONN_01X01" H 1250 6800 50  0000 C CNN
-F 2 "Socket_Strips:Socket_Strip_Straight_1x02" H 1250 6950 60  0001 C CNN
+F 2 "Pin_Headers:Pin_Header_Straight_1x01" H 1250 6950 60  0001 C CNN
 F 3 "" H 1250 6950 60  0000 C CNN
 	1    1250 6950
@@
 F 0 "P4" H 1250 7500 50  0000 C CNN
 F 1 "CONN_01X01" H 1250 7250 50  0000 C CNN
-F 2 "Socket_Strips:Socket_Strip_Straight_1x02" H 1250 7400 60  0001 C CNN
+F 2 "Pin_Headers:Pin_Header_Straight_1x01" H 1250 7400 60  0001 C CNN
 F 3 "" H 1250 7400 60  0000 C CNN
 	1    1250 7400
@@
 F 0 "P10" H 2100 6900 50  0000 C CNN
 F 1 "CONN_01X01" H 2100 6650 50  0000 C CNN
-F 2 "pcb:bornera_grande" H 2100 6800 60  0001 C CNN
+F 2 "Pin_Headers:Pin_Header_Straight_1x01" H 2100 6800 60  0001 C CNN
 F 3 "" H 2100 6800 60  0000 C CNN
 	1    2100 6800
@@
 F 0 "P9" H 2100 6200 50  0000 C CNN
 F 1 "CONN_01X01" H 2100 5950 50  0000 C CNN
-F 2 "pcb:bornera_grande" H 2100 6100 60  0001 C CNN
+F 2 "Pin_Headers:Pin_Header_Straight_1x01" H 2100 6100 60  0001 C CNN
 F 3 "" H 2100 6100 60  0000 C CNN
 	1    2100 6100
@@
 	2400 6100 2400 6150
 $Comp
-L Jack_3.5mm_5pin J?
+L Jack_3.5mm_5pin J1
 U 1 1 557AAF8F
 P 3000 2550
-F 0 "J?" H 3000 2800 60  0000 C CNN
+F 0 "J1" H 3000 2800 60  0000 C CNN
 F 1 "Jack_3.5mm_5pin" H 3000 2250 60  0000 C CNN
-F 2 "" H 3000 2600 60  0000 C CNN
+F 2 "pcb:jack_puto" H 3000 2600 60  0001 C CNN
 F 3 "" H 3000 2600 60  0000 C CNN
 	1    3000 2550
@@
 Connection ~ 2600 2350
 Wire Wire Line
-	2600 2450 2400 2450
-Wire Wire Line
-	2400 2450 2400 2750
-Wire Wire Line
-	2400 2750 2850 2750
-Wire Wire Line
-	2750 2750 2750 2650
-Wire Wire Line
 	2750 2650 2850 2650
-Connection ~ 2750 2750
-Wire Wire Line
-	2850 2550 2600 2550
-Wire Wire Line
-	2850 2450 2800 2450
-Wire Wire Line
-	2800 2450 2800 2550
-Connection ~ 2800 2550
+NoConn ~ 2850 2450
+$Comp
+L GND #PWR037
+U 1 1 557AC041
+P 2800 2900
+F 0 "#PWR037" H 2800 2650 50  0001 C CNN
+F 1 "GND" H 2800 2750 50  0000 C CNN
+F 2 "" H 2800 2900 60  0000 C CNN
+F 3 "" H 2800 2900 60  0000 C CNN
+	1    2800 2900
+	1    0    0    -1
+$EndComp
+Wire Wire Line
+	2800 2900 2800 2750
+Wire Wire Line
+	2500 2750 2850 2750
+Wire Wire Line
+	2850 2550 2500 2550
+Wire Wire Line
+	2500 2550 2500 2750
+Connection ~ 2800 2750
 $EndSCHEMATC

Commit message: Arreglando PCB
Parts:
- added R31, R32: R, Resistors_ThroughHole:Resistor_Horizontal_RM10mm, symbol R
Connections:
- net +VA: now also R13.1, R32.1; no longer Q11.1 (E), Q4.1 (E)
- net GND: now also R31.2; no longer R13.2
- net at Q4.2 (B), Q6.3 (C), R9.1: no longer Q6.2 (B)
- net at Q11.2 (B), Q9.3 (C): now also R31.1; no longer Q9.2 (B), R13.1
- new net: Q6.2 (B), R13.2
- new net: Q9.2 (B), R32.2
Other:
- moved on the sheet: Q4
