File: pcb/amplificador_gclass.kicad_pcb (KiCad board)
At the start: 2 copper layers, 163.8 x 63.5 mm, 88 parts, among them CON1 AUDIO_IN, P1 +VA_GND, P10 2SC3281, P11 2SC3281, P12 2SA1302, P2 +VB_GND, P3 -VA_GND, P4 -VB_GND, P5 OUT, P6 CONN_01X01, P7 MJE350, P8 MJE340, P9 2SA1302, Q1 MPSA56_PNP_EBC, Q10 MPSA06_NPN_EBC, Q11 MPSA56_PNP_EBC, Q12 MPSA06_NPN_EBC, Q13 MPSA56_PNP_EBC, Q14 MPSA06_NPN_EBC, Q15 MPSA56_PNP_EBC, Q16 MPSA06_NPN_EBC, Q17 MJE340_NPN_ECB, Q18 MJE350_PNP_EBC, Q19 MJE340_NPN_ECB, Q2 MPSA56_PNP_EBC, Q20 MJE350_PNP_EBC, Q3 MPSA06_NPN_EBC, Q4 MPSA56_PNP_EBC, Q5 MPSA06_NPN_EBC, Q6 MPSA56_PNP_EBC, Q7 MPSA56_PNP_EBC, Q8 MPSA56_PNP_EBC, Q9 MPSA56_PNP_EBC

Commit message: nacho la soba
Parts:
- P6: footprint Pin_Headers:Pin_Header_Straight_1x03 -> Pin_Headers:Pin_Header_Straight_1x01
- P7, P8: footprint Pin_Headers:Pin_Header_Straight_1x03 -> pcb:bornera_chica
- moved P10 123.0 mm to (119.6, -28.7)
- moved P11 123.0 mm to (136.0, 35.4)
- moved P12 123.0 mm to (127.9, 47.3)
- moved P9 123.0 mm to (123.6, 5.33)
- moved R27 123.0 mm to (146.7, -30.1)
- moved R28 123.0 mm to (147.1, 5.11)
- moved Q16 50.7 mm to (178.4, 118.3)
- moved Q14 50.7 mm to (172.0, 118.4)
- moved R21 50.2 mm to (179.4, 105.5)
- moved R18 50.2 mm to (179.2, 94.2)
- moved R20 50.2 mm to (179.2, 99.6)
- moved C11 48.6 mm to (217.5, 116.9)
- moved C13 48.6 mm to (197.0, 77.2)
- moved C15 48.6 mm to (209.9, 85.5)
- moved L1 48.6 mm to (228.8, 93.3)
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Connections:
- C15 pad 2: (no net) -> Net-(C15-Pad2)
- C3 pad 1: (no net) -> GND
Routing:
- net +VA: track 227.8 -> 47.4 mm
- net -VA: track 140.1 -> 21.5 mm
- net (no net): track 94.1 -> 0.50 mm, vias 2 -> 0
- net Net-(C8-Pad2): track 5.62 -> 73.9 mm
- net Net-(Q7-Pad2): track 109.8 -> 42.7 mm
- net Net-(D6-Pad1): track 66.0 -> 0.00 mm, vias 2 -> 0
- net Net-(P8-Pad3): track 62.8 -> 0.00 mm
- net TO_OPS: track 89.6 -> 29.7 mm
- net Net-(C9-Pad2): track 58.7 -> 0.36 mm
- net FBACK: track 57.8 -> 0.57 mm
- net Net-(P11-Pad1): track 50.4 -> 0.00 mm
- net +VB: track 49.6 -> 0.00 mm, vias 2 -> 0
- net Net-(P10-Pad1): track 47.8 -> 0.29 mm, vias 2 -> 0
- net Net-(P7-Pad3): track 47.3 -> 0.56 mm
- net Net-(C9-Pad1): track 38.6 -> 0.00 mm
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
Commit message: ultimos avances falta poco para terminar
Parts:
- removed R31: R, Resistors_ThroughHole:Resistor_Horizontal_RM10mm
- moved P9 132.4 mm to (184.5, 122.9), turned to 180 degrees
- moved R27 131.7 mm to (184.9, 95.9), turned to 90 degrees
- moved P10 104.6 mm to (151.3, 71.0), turned to 0 degrees
- moved R28 94.4 mm to (172.9, 95.9)
- moved Q20 87.1 mm to (117.0, 122.4), turned to 0 degrees
- moved R26 80.3 mm to (131.4, 123.5), turned to 180 degrees
- moved P12 76.8 mm to (142.4, 122.8)
- moved P11 64.7 mm to (190.0, 71.0)
- moved D4 63.3 mm to (123.4, 118.4)
- moved Q14 62.0 mm to (110.9, 107.6), turned to 180 degrees
- moved Q16 61.8 mm to (116.8, 113.5), turned to 0 degrees
- moved D5 52.2 mm to (163.3, 114.6)
- moved D3 52.0 mm to (120.7, 68.1), turned to 270 degrees
- moved R17 50.9 mm to (107.8, 116.4), turned to 270 degrees
- moved D2 49.7 mm to (134.8, 113.0), turned to 180 degrees
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Connections:
- C15 pad 2: Net-(C15-Pad2) -> GND
- P10 pad 1: Net-(P10-Pad1) -> Net-(C10-Pad1)
- P9 pad 1: Net-(P9-Pad1) -> Net-(C10-Pad2)
- Q17 pad 1: Net-(P10-Pad1) -> Net-(C10-Pad1)
- Q18 pad 1: Net-(P9-Pad1) -> Net-(C10-Pad2)
- R23 pad 1: Net-(C10-Pad1) -> Net-(R23-Pad1)
- R23 pad 2: Net-(P10-Pad1) -> Net-(C10-Pad1)
- R24 pad 1: Net-(C10-Pad2) -> Net-(R23-Pad1)
- R24 pad 2: Net-(P9-Pad1) -> Net-(C10-Pad2)
- R29 pad 2: GND -> Net-(C15-Pad1)
- R30 pad 1: FBACK -> OUT
- R30 pad 2: Net-(C15-Pad1) -> FBACK
Routing:
- net -VA: track 21.5 -> 241.7 mm
- net +VA: track 47.4 -> 201.5 mm
- net Net-(Q7-Pad2): track 42.7 -> 183.2 mm, vias 0 -> 2
- net FBACK: track 0.57 -> 110.7 mm, vias 0 -> 2
- net GND: track 0.00 -> 99.6 mm, vias 0 -> 2
- net Net-(P11-Pad1): track 0.00 -> 70.8 mm
- net Net-(C10-Pad2): track 0.07 -> 67.6 mm
- net Net-(C9-Pad1): track 0.00 -> 57.5 mm
- net -VB: track 0.00 -> 56.5 mm
- net Net-(C10-Pad1): track 0.05 -> 56.1 mm
- net +VB: track 0.00 -> 48.2 mm
- net Net-(D5-Pad2): track 0.42 -> 45.7 mm
- net Net-(C9-Pad2): track 0.36 -> 38.5 mm
- net Net-(P8-Pad3): track 0.00 -> 32.9 mm
- net Net-(P12-Pad1): track 0.00 -> 31.4 mm
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- added copper zone on B.Cu, net GND
Other:
- board size 163.8 x 63.5 mm -> 199.5 x 70.5 mm

Commit message: pcb casi listo
el pcb esta casi listo
Parts:
- added P13: CONN_01X01, Pin_Headers:Pin_Header_Straight_1x01, F.Cu at (78.5, 66.5)
- added P14: CONN_01X01, Pin_Headers:Pin_Header_Straight_1x01, F.Cu at (96.0, 66.5)
- added P15: CONN_01X01, Pin_Headers:Pin_Header_Straight_1x01, F.Cu at (30.5, 113.0)
- added P16: CONN_01X01, Pin_Headers:Pin_Header_Straight_1x01, F.Cu at (219.0, 75.0)
- added P17: CONN_01X01, Pin_Headers:Pin_Header_Straight_1x01, F.Cu at (222.0, 116.5)
- added P18: CONN_01X01, Pin_Headers:Pin_Header_Straight_1x01, F.Cu at (57.0, 67.0)
- added REF**: 1pin, Connect:1pin, F.Cu at (222.0, 67.5)
- added REF**: 1pin, Connect:1pin, F.Cu at (222.0, 130.0)
- added REF**: 1pin, Connect:1pin, F.Cu at (30.5, 130.0)
- added REF**: 1pin, Connect:1pin, F.Cu at (30.5, 67.5)
Routing:
- net GND: track 99.6 -> 394.0 mm
- net -VA: track 241.7 -> 246.3 mm
Other:
- net class Default: trace_width 0.381 -> 0.635
