File: pcb/amplificador_gclass.kicad_pcb (KiCad board)
At the start: 2 copper layers, 193.7 x 86.2 mm, 98 parts, among them J1 Jack_3.5mm_5pin, P1 CONN_01X01, P10 CONN_01X01, P12 OUT, P13 CONN_01X01, P14 MJE350, P15 MJE340, P16 2SA1302, P17 2SC3281, P18 2SC3281, P19 2SA1302, P2 CONN_01X01, P3 CONN_01X01, P4 CONN_01X01, P5 CONN_01X01, P6 CONN_01X01, P7 CONN_01X01, P8 CONN_01X01, P9 CONN_01X01, Q1 MPSA56_PNP_EBC, Q10 MPSA06_NPN_EBC, Q11 MPSA56_PNP_EBC, Q12 MPSA06_NPN_EBC, Q13 MPSA06_NPN_EBC, Q14 MPSA56_PNP_EBC, Q15 MPSA56_PNP_EBC, Q16 MPSA06_NPN_EBC, Q17 MJE340_NPN_ECB, Q18 MJE350_PNP_EBC, Q19 MJE340_NPN_ECB, Q2 MPSA56_PNP_EBC, Q20 MJE350_PNP_EBC, Q3 MPSA06_NPN_EBC, Q4 MPSA56_PNP_EBC, Q5 MPSA06_NPN_EBC, Q6 MPSA56_PNP_EBC, Q7 MPSA56_PNP_EBC, Q8 MPSA56_PNP_EBC, Q9 MPSA56_PNP_EBC

Commit message: algun cambio
Connections:
- Q11 pad 1: (no net) -> Net-(Q11-Pad1)
- Q4 pad 1: (no net) -> Net-(Q4-Pad1)
- Q6 pad 2: Net-(Q6-Pad2) -> Net-(Q4-Pad1)
- Q9 pad 2: Net-(Q9-Pad2) -> Net-(Q11-Pad1)
- R13 pad 1: +VA -> (no net)
- R13 pad 2: Net-(Q6-Pad2) -> Net-(Q4-Pad1)
- R32 pad 2: Net-(Q9-Pad2) -> Net-(Q11-Pad1)
Routing:
- net Net-(Q9-Pad2): track 15.2 -> 0.00 mm
- net Net-(Q11-Pad1): track 0.00 -> 15.2 mm
- net Net-(Q6-Pad2): track 4.23 -> 0.00 mm
- net Net-(Q4-Pad1): track 0.00 -> 4.23 mm
