File: pcb/$OPS.sch (KiCad schematic (older format))
At the start: 44 parts, among them P14 MJE350, P15 MJE340, P16 2SA1302, P17 2SC3281, P18 2SC3281, P19 2SA1302, Q13 MPSA56_PNP_EBC, Q14 MPSA06_NPN_EBC, Q15 MPSA56_PNP_EBC, Q16 MPSA06_NPN_EBC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

Commit message: pcb terminado
Parts:
- P14, P15: footprint Pin_Headers:Pin_Header_Straight_1x01 -> pcb:bornera_chica
- P16, P17, P18: footprint Pin_Headers:Pin_Header_Straight_1x01 -> pcb:bornera_grande
Changed lines of the file:
@@
 LIBS:contrib
 LIBS:valves
+LIBS:w_connectors
 LIBS:amplificador_gclass-cache
 EELAYER 25 0
@@
 F 0 "P14" H 3850 3350 50  0000 C CNN
 F 1 "MJE350" V 3950 3150 50  0000 C CNN
-F 2 "Pin_Headers:Pin_Header_Straight_1x01" H 3850 3150 60  0001 C CNN
+F 2 "pcb:bornera_chica" H 3850 3150 60  0001 C CNN
 F 3 "" H 3850 3150 60  0000 C CNN
 	1    3850 3150
@@
 F 0 "P15" H 3850 4050 50  0000 C CNN
 F 1 "MJE340" V 3950 3850 50  0000 C CNN
-F 2 "Pin_Headers:Pin_Header_Straight_1x01" H 3850 3850 60  0001 C CNN
+F 2 "pcb:bornera_chica" H 3850 3850 60  0001 C CNN
 F 3 "" H 3850 3850 60  0000 C CNN
 	1    3850 3850
@@
 F 0 "P17" H 5550 2950 50  0000 C CNN
 F 1 "2SC3281" V 5650 2750 50  0000 C CNN
-F 2 "Pin_Headers:Pin_Header_Straight_1x01" H 5550 2750 60  0001 C CNN
+F 2 "pcb:bornera_grande" H 5550 2750 60  0001 C CNN
 F 3 "" H 5550 2750 60  0000 C CNN
 	1    5550 2750
@@
 F 0 "P16" H 5450 4050 50  0000 C CNN
 F 1 "2SA1302" V 5550 3850 50  0000 C CNN
-F 2 "Pin_Headers:Pin_Header_Straight_1x01" H 5450 3850 60  0001 C CNN
+F 2 "pcb:bornera_grande" H 5450 3850 60  0001 C CNN
 F 3 "" H 5450 3850 60  0000 C CNN
 	1    5450 3850
@@
 F 0 "P18" H 6300 2150 50  0000 C CNN
 F 1 "2SC3281" V 6400 1950 50  0000 C CNN
-F 2 "Pin_Headers:Pin_Header_Straight_1x01" H 6300 1950 60  0001 C CNN
+F 2 "pcb:bornera_grande" H 6300 1950 60  0001 C CNN
 F 3 "" H 6300 1950 60  0000 C CNN
 	1    6300 1950
