File: pcb/$amplificador_gclass.sch (KiCad schematic (older format))
At the start: 51 parts, among them J1 Jack_3.5mm_5pin, P1 CONN_01X01, P10 CONN_01X01, P12 OUT, P13 CONN_01X01, P2 CONN_01X01, P3 CONN_01X01, P4 CONN_01X01, P5 CONN_01X01, P6 CONN_01X01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

Commit message: Cambio las fuentes de corrientes por unas mas estables, agrando todas las pistas, agrego mini planos de tension para potencia, cambio pines de salida.
Parts:
- P5, P6, P7, P8: footprint Pin_Headers:Pin_Header_Straight_1x02 -> Pin_Headers:Pin_Header_Straight_1x01
Changed lines of the file:
@@
 F 0 "P5" H 1400 2450 50  0000 C CNN
 F 1 "CONN_01X01" V 1500 2350 50  0000 C CNN
-F 2 "Pin_Headers:Pin_Header_Straight_1x02" H 1400 2350 60  0001 C CNN
+F 2 "Pin_Headers:Pin_Header_Straight_1x01" H 1400 2350 60  0001 C CNN
 F 3 "" H 1400 2350 60  0000 C CNN
 	1    1400 2350
@@
 F 0 "P7" H 1950 2450 50  0000 C CNN
 F 1 "CONN_01X01" V 2050 2350 50  0000 C CNN
-F 2 "Pin_Headers:Pin_Header_Straight_1x02" H 1950 2350 60  0001 C CNN
+F 2 "Pin_Headers:Pin_Header_Straight_1x01" H 1950 2350 60  0001 C CNN
 F 3 "" H 1950 2350 60  0000 C CNN
 	1    1950 2350
@@
 F 0 "P6" H 1400 3350 50  0000 C CNN
 F 1 "CONN_01X01" V 1500 3250 50  0000 C CNN
-F 2 "Pin_Headers:Pin_Header_Straight_1x02" H 1400 3250 60  0001 C CNN
+F 2 "Pin_Headers:Pin_Header_Straight_1x01" H 1400 3250 60  0001 C CNN
 F 3 "" H 1400 3250 60  0000 C CNN
 	1    1400 3250
@@
 F 0 "P8" H 1950 3350 50  0000 C CNN
 F 1 "CONN_01X01" V 2050 3250 50  0000 C CNN
-F 2 "Pin_Headers:Pin_Header_Straight_1x02" H 1950 3250 60  0001 C CNN
+F 2 "Pin_Headers:Pin_Header_Straight_1x01" H 1950 3250 60  0001 C CNN
 F 3 "" H 1950 3250 60  0000 C CNN
 	1    1950 3250
