File: pcb/amplificador.kicad_pcb (KiCad board)
At the start: 2 copper layers, 92 parts, among them Q1 2SC3281, Q10 MPSA42, Q11 2SC3281, Q12 2SA1302, Q13 MPSA92, Q14 MPSA92, Q15 MJE340, Q16 MJE350, Q17 MJE350, Q2 MJE340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

Commit message: asht
Routing:
- net SalidaGND: track 480.5 -> 462.7 mm
- net (no net): track 0.00 -> 17.8 mm
Changed lines of the file:
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@@
-(kicad_pcb (version 20170123) (host pcbnew "(2017-02-08 revision 0dc11936a)-master")
+(kicad_pcb (version 4) (host pcbnew 4.0.2-stable)
   (general
     (links 166)
-    (no_connects 1)
-    (area 45 16 227.4565 157.000001)
+    (no_connects 0)
+    (area 45 16 227.339 157.000001)
     (thickness 1.6)
     (drawings 2)
@@
   (layers
     (0 F.Cu signal)
-    (31 B.Cu signal)
+    (31 B.Cu signal hide)
     (32 B.Adhes user)
     (33 F.Adhes user)
@@
     (45 Margin user)
     (46 B.CrtYd user)
-    (47 F.CrtYd user)
+    (47 F.CrtYd user hide)
     (48 B.Fab user)
     (49 F.Fab user)
@@
     (pad_to_mask_clearance 0)
     (aux_axis_origin 0 0)
-    (visible_elements FFFFFF7F)
+    (visible_elements FFFEEF7F)
     (pcbplotparams
       (layerselection 0x01000_ffffffff)
@@
       (hpglpenspeed 20)
       (hpglpendiameter 15)
+      (hpglpenoverlay 2)
       (psnegative false)
       (psa4output false)
@@
     (effects (font (size 1.5 1.5) (thickness 0.3)))
   )
+  (segment (start 70 53) (end 72 51) (width 0.5) (layer F.Cu) (net 0))
+  (segment (start 55 53) (end 70 53) (width 0.5) (layer F.Cu) (net 0))
   (segment (start 77.586 77.5) (end 77.586 73.16) (width 1) (layer B.Cu) (net 1))
   (segment (start 57.409 102.983) (end 66.796 102.983) (width 0.65) (layer F.Cu) (net 2))
@@
   (segment (start 59.386 58.16) (end 55.226 54) (width 1) (layer B.Cu) (net 61))
   (via (at 55.226 54) (size 0.8) (drill 0.4) (layers F.Cu B.Cu) (net 61))
-  (segment (start 70 53) (end 72 51) (width 0.5) (layer F.Cu) (net 61))
-  (segment (start 55 53) (end 70 53) (width 0.5) (layer F.Cu) (net 61))
   (segment (start 59.386 58.16) (end 62.086 60.86) (width 0.5) (layer F.Cu) (net 61))
   (segment (start 62.086 60.86) (end 62.086 65.66) (width 0.5) (layer F.Cu) (net 61))
